File: Projects/Tutorial01/Tutorial01.kicad_sch (KiCad schematic)
At the start: 4 parts

Commit message: 20251113 Schaltplan mit Batterie 9V, eine rote Diode 3 mm Durchmnesser und ein Widerstand 220 ohm
Parts:
- removed R2: R, symbol Device:R
- Batterie1: renamed from Batterie; footprint (none) -> Battery:BatteryHolder_Keystone_103_1x20mm
- D1: footprint (none) -> LED_THT:LED_D3.0mm
- R1: footprint (none) -> Resistor_THT:R_Axial_DIN0207_L6.3mm_D2.5mm_P10.16mm_Horizontal
Changed lines of the file:
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@@
 			)
 		)
-		(property "Footprint" ""
+		(property "Footprint" "LED_THT:LED_D3.0mm"
 			(at 68.58 74.93 0)
 			(effects
@@
 		(dnp no)
 		(fields_autoplaced yes)
-		(property "Reference" "Batterie"
+		(property "Reference" "Batterie1"
 			(at 64.77 81.9784 0)
 			(effects
@@
 			)
 		)
-		(property "Footprint" ""
+		(property "Footprint" "Battery:BatteryHolder_Keystone_103_1x20mm"
 			(at 60.96 82.296 90)
 			(effects
@@
 			(project ""
 				(path "/8ae59741-537a-42c7-8cdd-92d8d9dc48c6"
-					(reference "Batterie")
+					(reference "Batterie1")
 					(unit 1)
 				)
@@
 			)
 		)
-		(property "Footprint" ""
+		(property "Footprint" "Resistor_THT:R_Axial_DIN0207_L6.3mm_D2.5mm_P10.16mm_Horizontal"
 			(at 80.01 76.708 90)
 			(effects
@@
 					(unit 1)
 				)
-			)
-		)
-	)
-	(symbol
-		(lib_id "Device:R")
-		(at 90.17 100.33 0)
-		(unit 1)
-		(exclude_from_sim no)
-		(in_bom yes)
-		(on_board yes)
-		(dnp no)
-		(fields_autoplaced yes)
-		(property "Reference" "R2"
-			(at 92.71 99.0599 0)
-			(effects
-				(font
-					(size 1.27 1.27)
-				)
-				(justify left)
-			)
-		)
-		(property "Value" "R"
-			(at 92.71 101.5999 0)
-			(effects
-				(font
-					(size 1.27 1.27)
-				)
-				(justify left)
-			)
-		)
-		(property "Footprint" ""
-			(at 88.392 100.33 90)
-			(effects
-				(font
-					(size 1.27 1.27)
-				)
-				(hide yes)
-			)
-		)
-		(property "Datasheet" "~"
-			(at 90.17 100.33 0)
-			(effects
-				(font
-					(size 1.27 1.27)
-				)
-				(hide yes)
-			)
-		)
-		(property "Description" "Resistor"
-			(at 90.17 100.33 0)
-			(effects
-				(font
-					(size 1.27 1.27)
-				)
-				(hide yes)
-			)
-		)
-		(pin "1"
-		)
-		(pin "2"
-		)
-		(instances
-			(project ""
-				(path "/8ae59741-537a-42c7-8cdd-92d8d9dc48c6"
-					(reference "R2")
-					(unit 1)
-				)
