File: Projects/Tutorial02/Tutorial02.kicad_sch (KiCad schematic)
At the start: 16 parts, among them J1 FTDI Programmer, J2 Arduino PIN0 - PIN7, J3 Arduino A0 - A5, J4 Power & Ground Terminal, J5 Versorgungsspannung, J6 Arduino PIN8 - PIN13, U1 ATMEGA328P-PU, Y1 Crystal

Commit message: 20251206 tutorial02
Other:
- note added: "Arduino PIN A0"
- note added: "Arduino PIN A1"
- note added: "Arduino PIN A2"
- note added: "Arduino PIN A3"
- note added: "Arduino PIN A4"
- note added: "Arduino PIN A5"
- moved on the sheet: J1, J3, J4
Changed lines of the file:
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@@
 	(text "RX"
 		(exclude_from_sim no)
-		(at 89.408 49.53 0)
+		(at 90.678 48.26 0)
+		(effects
+			(font
+				(size 1.27 1.27)
+			)
+		)
+	)
+	(text "GND"
+		(exclude_from_sim no)
+		(at 92.202 156.464 0)
 		(effects
 			(font
@@
 	(text "DTR"
 		(exclude_from_sim no)
-		(at 89.408 54.864 0)
+		(at 90.678 53.594 0)
+		(effects
+			(font
+				(size 1.27 1.27)
+			)
+		)
+	)
+	(text "Arduino PIN A0\n"
+		(exclude_from_sim no)
+		(at 87.376 129.54 0)
+		(effects
+			(font
+				(size 1.27 1.27)
+			)
+		)
+	)
+	(text "Arduino PIN A5\n"
+		(exclude_from_sim no)
+		(at 87.376 116.84 0)
+		(effects
+			(font
+				(size 1.27 1.27)
+			)
+		)
+	)
+	(text "Arduino PIN A4\n"
+		(exclude_from_sim no)
+		(at 87.376 119.634 0)
+		(effects
+			(font
+				(size 1.27 1.27)
+			)
+		)
+	)
+	(text "Arduino PIN A2\n"
+		(exclude_from_sim no)
+		(at 87.376 124.46 0)
 		(effects
 			(font
@@
 	(text "GND"
 		(exclude_from_sim no)
-		(at 89.408 57.404 0)
+		(at 90.932 56.134 0)
 		(effects
 			(font
@@
 	(text "TX"
 		(exclude_from_sim no)
-		(at 89.662 52.324 0)
+		(at 90.932 51.054 0)
+		(effects
+			(font
+				(size 1.27 1.27)
+			)
+		)
+	)
+	(text "GND"
+		(exclude_from_sim no)
+		(at 92.202 153.924 0)
+		(effects
+			(font
+				(size 1.27 1.27)
+			)
+		)
+	)
+	(text "Arduino PIN A3\n"
+		(exclude_from_sim no)
+		(at 87.376 122.174 0)
+		(effects
+			(font
+				(size 1.27 1.27)
+			)
+		)
+	)
+	(text "GND"
+		(exclude_from_sim no)
+		(at 92.202 151.384 0)
 		(effects
 			(font
@@
 	(text "5 V"
 		(exclude_from_sim no)
-		(at 89.154 46.99 0)
+		(at 90.424 45.72 0)
+		(effects
+			(font
+				(size 1.27 1.27)
+			)
+		)
+	)
+	(text "Arduino PIN A1\n"
+		(exclude_from_sim no)
+		(at 87.376 127 0)
 		(effects
 			(font
@@
 		(lib_id "Connector:Conn_01x06_Pin")
 		(at 95.25 124.46 0)
+		(mirror x)
 		(unit 1)
 		(exclude_from_sim no)
@@
 		(dnp no)
 		(property "Reference" "J3"
-			(at 85.09 114.3 0)
+			(at 85.09 112.522 0)
 			(effects
 				(font
@@
 		)
 		(property "Value" "Arduino A0 - A5"
-			(at 95.25 114.554 0)
+			(at 95.25 112.268 0)
 			(effects
 				(font
@@
 		(dnp no)
 		(property "Reference" "J6"
-			(at 86.106 88.138 0)
+			(at 82.042 88.138 0)
 			(effects
 				(font
@@
 		)
 		(property "Value" "Arduino PIN8 - PIN13"
-			(at 99.314 88.138 0)
+			(at 95.25 88.138 0)
 			(effects
 				(font
@@
 		(lib_id "Connector:Conn_01x06_Pin")
 		(at 95.25 151.13 0)
+		(mirror x)
 		(unit 1)
 		(exclude_from_sim no)
@@
 		(dnp no)
 		(property "Reference" "J4"
-			(at 84.836 140.97 0)
+			(at 81.026 138.43 0)
 			(effects
 				(font
@@
 		)
 		(property "Value" "Power & Ground Terminal"
-			(at 99.06 140.97 0)
+			(at 95.25 138.43 0)
 			(effects
 				(font
@@
 		(dnp no)
 		(property "Reference" "J2"
-			(at 86.868 61.214 0)
+			(at 81.28 61.214 0)
 			(effects
 				(font
@@
 		)
 		(property "Value" "Arduino PIN0 - PIN7"
-			(at 99.314 60.96 0)
+			(at 93.726 60.96 0)
 			(effects
 				(font
@@
 	(symbol
 		(lib_id "Connector:Conn_01x05_Pin")
-		(at 92.71 52.07 0)
+		(at 93.98 50.8 0)
 		(unit 1)
 		(exclude_from_sim no)
@@
 		(dnp no)
 		(property "Reference" "J1"
-			(at 85.09 42.164 0)
+			(at 84.074 40.894 0)
 			(effects
 				(font
@@
 		)
 		(property "Value" "FTDI Programmer"
-			(at 94.996 42.164 0)
+			(at 93.98 40.894 0)
 			(effects
 				(font
@@
 		)
 		(property "Footprint" ""
-			(at 92.71 52.07 0)
+			(at 93.98 50.8 0)
 			(effects
 				(font
@@
 		)
 		(property "Datasheet" "~"
-			(at 92.71 52.07 0)
+			(at 93.98 50.8 0)
 			(effects
 				(font
@@
 		)
 		(property "Description" "Generic connector, single row, 01x05, script generated"
-			(at 92.71 52.07 0)
-			(effects
-				(font
+			(at 93.98 50.8 0)
+			(effects
+				(font

Commit message: 20251206 tutorial02
Other:
- note added: "Arduino PIN 0"
Changed lines of the file:
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@@
 		(comment 1 "Designed by Davide Spano")
 	)
+	(text "Arduino PIN 0\n"
+		(exclude_from_sim no)
+		(at 87.122 103.124 0)
+		(effects
+			(font
+				(size 1.27 1.27)
+			)
+		)
+	)
 	(text "RX"
 		(exclude_from_sim no)
@@
 		)
 	)
+	(text "5 V\n"
+		(exclude_from_sim no)
+		(at 92.202 146.304 0)
+		(effects
+			(font
+				(size 1.27 1.27)
+			)
+		)
+	)
+	(text "Arduino PIN 0\n"
+		(exclude_from_sim no)
+		(at 87.122 95.504 0)
+		(effects
+			(font
+				(size 1.27 1.27)
+			)
+		)
+	)
+	(text "Arduino PIN 0\n"
+		(exclude_from_sim no)
+		(at 85.852 72.644 0)
+		(effects
+			(font
+				(size 1.27 1.27)
+			)
+		)
+	)
 	(text "DTR"
 		(exclude_from_sim no)
@@
 		)
 	)
+	(text "5 V\n"
+		(exclude_from_sim no)
+		(at 92.202 148.844 0)
+		(effects
+			(font
+				(size 1.27 1.27)
+			)
+		)
+	)
 	(text "Arduino PIN A0\n"
 		(exclude_from_sim no)
@@
 		)
 	)
+	(text "5 V\n"
+		(exclude_from_sim no)
+		(at 92.202 143.764 0)
+		(effects
+			(font
+				(size 1.27 1.27)
+			)
+		)
+	)
 	(text "Arduino PIN A4\n"
 		(exclude_from_sim no)
@@
 		)
 	)
+	(text "Arduino PIN 0\n"
+		(exclude_from_sim no)
+		(at 87.122 100.584 0)
+		(effects
+			(font
+				(size 1.27 1.27)
+			)
+		)
+	)
+	(text "Arduino PIN 0\n"
+		(exclude_from_sim no)
+		(at 85.852 80.264 0)
+		(effects
+			(font
+				(size 1.27 1.27)
+			)
+		)
+	)
 	(text "TX"
 		(exclude_from_sim no)
@@
 		)
 	)
+	(text "Arduino PIN 0\n"
+		(exclude_from_sim no)
+		(at 85.852 65.024 0)
+		(effects
+			(font
+				(size 1.27 1.27)
+			)
+		)
+	)
 	(text "GND"
 		(exclude_from_sim no)
@@
 		)
 	)
+	(text "Arduino PIN 0\n"
+		(exclude_from_sim no)
+		(at 85.852 77.47 0)
+		(effects
+			(font
+				(size 1.27 1.27)
+			)
+		)
+	)
+	(text "Arduino PIN 0\n"
+		(exclude_from_sim no)
+		(at 87.122 98.044 0)
+		(effects
+			(font
+				(size 1.27 1.27)
+			)
+		)
+	)
+	(text "Arduino PIN 0\n"
+		(exclude_from_sim no)
+		(at 87.122 92.964 0)
+		(effects
+			(font
+				(size 1.27 1.27)
+			)
+		)
+	)
 	(text "Arduino PIN A3\n"
 		(exclude_from_sim no)
@@
 		)
 	)
+	(text "Arduino PIN 0\n"
+		(exclude_from_sim no)
+		(at 85.852 70.104 0)
+		(effects
+			(font
+				(size 1.27 1.27)
+			)
+		)
+	)
+	(text "Arduino PIN 0\n"
+		(exclude_from_sim no)
+		(at 87.122 105.664 0)
+		(effects
+			(font
+				(size 1.27 1.27)
+			)
+		)
+	)
+	(text "Arduino PIN 0\n"
+		(exclude_from_sim no)
+		(at 85.852 74.93 0)
+		(effects
+			(font
+				(size 1.27 1.27)
+			)
+		)
+	)
+	(text "Arduino PIN 0\n"
+		(exclude_from_sim no)
+		(at 85.852 82.804 0)
+		(effects
+			(font
+				(size 1.27 1.27)
+			)
+		)
+	)
 	(text "5 V"
 		(exclude_from_sim no)
@@
 		(effects
 			(font
+				(size 1.27 1.27)
+			)
+		)
+	)
+	(text "Arduino PIN 0\n"
+		(exclude_from_sim no)
+		(at 85.852 67.564 0)
+		(effects
+			(font

Commit message: 20251207 tutorial02
Other:
- note added: "Arduino PIN 1"
- note added: "Arduino PIN 10"
- note added: "Arduino PIN 11"
- note added: "Arduino PIN 12"
- note added: "Arduino PIN 13"
- note added: "Arduino PIN 2"
- note added: "Arduino PIN 3"
- note added: "Arduino PIN 4"
- note added: "Arduino PIN 5"
- note added: "Arduino PIN 6"
- note added: "Arduino PIN 7"
- note added: "Arduino PIN 8"
- note added: "Arduino PIN 9"
