File: Projects/Tutorial02/Tutorial02.kicad_sch (KiCad schematic)
At the start: 16 parts, among them J1 FTDI Programmer, J2 Arduino PIN0 - PIN7, J3 Arduino A0 - A5, J4 Power & Ground Terminal, J5 Versorgungsspannung, J6 Arduino PIN8 - PIN13, U1 ATMEGA328P-PU, Y1 Crystal

Commit message: 20251209 tutorial02
Connections:
- net GND: now also D1.1 (K), U1.22 (GND), U1.8 (GND)
- net at D1.2 (A): now also R3.2
- net RX: now reaches U1.2 (PD0)
- net RX: now also J1.3 (Pin_3)
- net TX: now reaches U1.3 (PD1)
- net TX: now also J1.2 (Pin_2)
Other:
- moved on the sheet: D1, R3

Commit message: 20251209 tutorial02
Connections:
- net +5V: now also J1.1 (Pin_1), U1.20 (AVCC), U1.7 (VCC)
- net GND: now also J1.4 (Pin_4), J1.5 (Pin_5), S1.1, S1.2
- net RESET: now reaches S1.3
- net RESET: now also S1.4, U1.1 (PC6)
Other:
- moved on the sheet: C1, C2, C3, C4, C5, D1, J1, J2, J3, J4, J5, J6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

Commit message: 20251210 tutorial02
Parts:
- added R1: 10K, symbol Device:R
- C1, C3: value C -> 100nF
- C4, C5: value C -> 22pF
Connections:
- net +5V: now also R1.2
- net GND: now also C1.1, C4.1, C5.1, R3.1; no longer D1.1 (K), J1.4 (Pin_4)
- net RESET: now also C3.2, R1.1
- net PC0: now reaches J3.1 (Pin_1)
- net PC0: now also U1.23 (PC0)
- net PC1: now reaches J3.2 (Pin_2)
- net PC1: now also U1.24 (PC1)
- net PC2: now reaches J3.3 (Pin_3)
- net PC2: now also U1.25 (PC2)
- net PC3: now reaches J3.4 (Pin_4)
- net PC3: now also U1.26 (PC3)
- net PC4: now reaches J3.5 (Pin_5)
- net PC4: now also U1.27 (PC4)
- net PC5: now reaches J3.6 (Pin_6)
- net PC5: now also U1.28 (PC5)
- net PB0: now reaches J6.1 (Pin_1)
- net PB0: now also U1.14 (PB0)
- net PB1: now reaches J6.2 (Pin_2)
- net PB1: now also U1.15 (PB1)
- net PB2: now reaches J6.3 (Pin_3)
- net PB2: now also U1.16 (PB2)
- net PB3: now reaches J6.4 (Pin_4)
- net PB3: now also U1.17 (PB3)
- net PB4: now reaches J6.5 (Pin_5)
- net PB4: now also U1.18 (PB4)
- net PB5: now reaches J6.6 (Pin_6)
- net PB5: now also D1.1 (K), U1.19 (PB5)
- net PD0: now reaches J2.1 (Pin_1)
- net PD1: now reaches J2.2 (Pin_2)
- net PD2: now reaches J2.3 (Pin_3)
- net PD2: now also U1.4 (PD2)
- net PD3: now reaches J2.4 (Pin_4)
- net PD3: now also U1.5 (PD3)
- net PD4: now reaches J2.5 (Pin_5)
- net PD4: now also U1.6 (PD4)
- net PD5: now reaches J2.6 (Pin_6)
- net PD5: now also U1.11 (PD5)
- net PD6: now reaches J2.7 (Pin_7)
- net PD6: now also U1.12 (PD6)
- net PD7: now reaches J2.8 (Pin_8)
- net PD7: now also U1.13 (PD7)
- net at C5.2: now also U1.9 (PB6), Y1.2
- net at C4.2: now also U1.10 (PB7), Y1.1
- net DTR: now reaches C3.1
- net DTR: now also J1.4 (Pin_4)
- net at U1.21 (AREF): now also C1.2
Other:
- moved on the sheet: C1, C3, C4, C5, D1, J1, R3, S1, Y1

Commit message: 20251212 tutorial02
Parts:
- C2: value C -> 100nF
Connections:
- net +5V: now also C2.1
- net GND: now also C2.2
Other:
- moved on the sheet: C1, C2, C3, C4, C5, D1, J1, J2, J3, J4, J5, J6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

Commit message: 20251212 tutorial02
Connections:
- net +5V: now also J4.4 (Pin_4), J4.5 (Pin_5), J4.6 (Pin_6)
- net GND: now also J4.1 (Pin_1), J4.2 (Pin_2), J4.3 (Pin_3)

Commit message: 20251212 tutorial02
Parts:
- C1, C2, C3: footprint (none) -> Capacitor_THT:C_Disc_D6.0mm_W2.5mm_P5.00mm
- C4, C5: footprint (none) -> Capacitor_THT:C_Disc_D3.8mm_W2.6mm_P2.50mm
- D1: footprint (none) -> LED_THT:LED_D5.0mm
- J1: footprint (none) -> Connector_PinHeader_2.54mm:PinHeader_1x05_P2.54mm_Vertical
- J2: footprint (none) -> Connector_PinHeader_2.54mm:PinHeader_1x08_P2.54mm_Vertical
- J3, J4, J6: footprint (none) -> Connector_PinHeader_2.54mm:PinHeader_1x06_P2.54mm_Vertical
- J5: footprint (none) -> TerminalBlock_TE-Connectivity:TerminalBlock_TE_282834-2_1x02_P2.54mm_Horizontal
- R1, R3: footprint (none) -> Resistor_THT:R_Axial_DIN0204_L3.6mm_D1.6mm_P7.62mm_Horizontal
- S1: footprint digikey-footprints:Switch_Tactile_THT_6x6mm -> Button_Switch_THT:SW_PUSH-12mm
- U1: footprint digikey-footprints:DIP-28_W7.62mm -> (none)
Changed lines of the file:
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@@
 			)
 		)
-		(property "Footprint" "digikey-footprints:Switch_Tactile_THT_6x6mm"
+		(property "Footprint" "Button_Switch_THT:SW_PUSH-12mm"
 			(at 137.16 48.26 0)
 			(effects
@@
 			)
 		)
-		(property "Footprint" ""
+		(property "Footprint" "Capacitor_THT:C_Disc_D6.0mm_W2.5mm_P5.00mm"
 			(at 204.47 51.1048 0)
 			(effects
@@
 			)
 		)
-		(property "Footprint" ""
+		(property "Footprint" "Connector_PinHeader_2.54mm:PinHeader_1x06_P2.54mm_Vertical"
 			(at 95.25 115.57 0)
 			(effects
@@
 			)
 		)
-		(property "Footprint" ""
+		(property "Footprint" "Connector_PinHeader_2.54mm:PinHeader_1x06_P2.54mm_Vertical"
 			(at 95.25 91.44 0)
 			(effects
@@
 			)
 		)
-		(property "Footprint" ""
+		(property "Footprint" "LED_THT:LED_D5.0mm"
 			(at 157.48 134.62 0)
 			(effects
@@
 			)
 		)
-		(property "Footprint" ""
+		(property "Footprint" "Connector_PinHeader_2.54mm:PinHeader_1x06_P2.54mm_Vertical"
 			(at 95.25 142.24 0)
 			(effects
@@
 			)
 		)
-		(property "Footprint" ""
+		(property "Footprint" "Connector_PinHeader_2.54mm:PinHeader_1x08_P2.54mm_Vertical"
 			(at 93.98 66.04 0)
 			(effects
@@
 			)
 		)
-		(property "Footprint" ""
+		(property "Footprint" "Capacitor_THT:C_Disc_D3.8mm_W2.6mm_P2.50mm"
 			(at 146.05 73.9648 0)
 			(effects
@@
 			)
 		)
-		(property "Footprint" ""
+		(property "Footprint" "Capacitor_THT:C_Disc_D3.8mm_W2.6mm_P2.50mm"
 			(at 146.05 84.1248 0)
 			(effects
@@
 			)
 		)
-		(property "Footprint" ""
+		(property "Footprint" "Capacitor_THT:C_Disc_D6.0mm_W2.5mm_P5.00mm"
 			(at 144.4752 46.99 0)
 			(effects
@@
 			)
 		)
-		(property "Footprint" ""
+		(property "Footprint" "Resistor_THT:R_Axial_DIN0204_L3.6mm_D1.6mm_P7.62mm_Horizontal"
 			(at 157.988 43.18 90)
 			(effects
@@
 			)
 		)
-		(property "Footprint" "digikey-footprints:DIP-28_W7.62mm"
+		(property "Footprint" ""
 			(at 198.12 86.36 0)
 			(effects
@@
 			)
 		)
-		(property "Footprint" ""
+		(property "Footprint" "Connector_PinHeader_2.54mm:PinHeader_1x05_P2.54mm_Vertical"
 			(at 91.44 41.91 0)
 			(effects
@@
 			)
 		)
-		(property "Footprint" ""
+		(property "Footprint" "Resistor_THT:R_Axial_DIN0204_L3.6mm_D1.6mm_P7.62mm_Horizontal"
 			(at 150.368 139.7 90)
 			(effects
@@
 			)
 		)
-		(property "Footprint" ""
+		(property "Footprint" "TerminalBlock_TE-Connectivity:TerminalBlock_TE_282834-2_1x02_P2.54mm_Horizontal"
 			(at 91.44 162.56 0)
 			(effects
@@
 			)
 		)
-		(property "Footprint" ""
+		(property "Footprint" "Capacitor_THT:C_Disc_D6.0mm_W2.5mm_P5.00mm"
 			(at 162.56 105.7148 0)
 			(effects

Commit message: 20251212 tutorial02
Parts:
- U1: footprint (none) -> Package_DIP:DIP-28_W7.62mm
- Y1: footprint (none) -> Crystal:Crystal_HC52-6mm_Vertical
Changed lines of the file:
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@@
 			)
 		)
-		(property "Footprint" ""
+		(property "Footprint" "Package_DIP:DIP-28_W7.62mm"
 			(at 198.12 86.36 0)
 			(effects
@@
 			)
 		)
-		(property "Footprint" ""
+		(property "Footprint" "Crystal:Crystal_HC52-6mm_Vertical"
 			(at 158.75 80.01 0)
 			(effects

Commit message: 20251220-tutorial-14
Parts:
- S1: footprint Button_Switch_THT:SW_PUSH-12mm -> Button_Switch_THT:SW_TH_Tactile_Omron_B3F-100x
Changed lines of the file:
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@@
 			)
 		)
-		(property "Footprint" "Button_Switch_THT:SW_PUSH-12mm"
+		(property "Footprint" "Button_Switch_THT:SW_TH_Tactile_Omron_B3F-100x"
 			(at 137.16 48.26 0)
 			(effects
