File: Projects/Tutorial02/Tutorial02.kicad_pcb (KiCad board)
At the start: 2 copper layers, 17 parts, among them J1 FTDI Programmer, J2 Arduino PIN0 - PIN7, J3 Arduino A0 - A5, J4 Power & Ground Terminal, J5 Versorgungsspannung, J6 Arduino PIN8 - PIN13, U1 ATMEGA328P-PU, Y1 Crystal

Commit message: 20251222-tutorial-15
Parts:
- removed S1: Reset, Button_Switch_THT:SW_TH_Tactile_Omron_B3F-100x
- added SW1: SW_Push, Button_Switch_THT:SW_PUSH_6mm_H7.3mm, F.Cu at (135.5, 77.0)
- moved C4 43.9 mm to (114.5, 111.5), turned to 180 degrees
- moved J4 43.7 mm to (114.0, 119.5), turned to 90 degrees
- moved J5 40.8 mm to (106.5, 74.5)
- moved J6 37.6 mm to (135.0, 118.5), turned to 180 degrees
- moved J1 37.6 mm to (106.5, 90.5), turned to 180 degrees
- moved C5 37.3 mm to (114.5, 98.5), turned to 180 degrees
- moved Y1 35.4 mm to (113.2, 106.8), turned to 90 degrees
- moved C3 30.6 mm to (125.5, 77.0), turned to 90 degrees
- moved C2 24.3 mm to (112.5, 91.5), turned to 90 degrees
- moved J2 24.0 mm to (106.5, 97.0)
- moved R1 23.6 mm to (120.0, 77.5), turned to 180 degrees
- moved D1 17.8 mm to (135.2, 100.5)
- moved J3 13.1 mm to (135.0, 93.5), turned to 180 degrees
- moved R3 5.80 mm to (138.5, 86.7), turned to -90 degrees
- moved C1 4.68 mm to (130.5, 95.5), turned to -90 degrees
Connections:
- net RESET renamed Net-(U1-PC6)

Commit message: 20251228
Parts:
- moved J4 1.00 mm to (114.0, 118.5)
Other:
- board outline added: 36.5 x 51 mm
Changed lines of the file:
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@@
 		(tags "Through hole pin header THT 1x08 2.54mm single row")
 		(property "Reference" "J2"
-			(at 0 -2.38 0)
+			(at 0 20.54 0)
 			(layer "F.SilkS")
 			(effects
@@
 		(tags "Resistor Axial_DIN0204 series Axial Horizontal pin pitch 7.62mm 0.167W length 3.6mm diameter 1.6mm")
 		(property "Reference" "R1"
-			(at 3.81 -1.92 0)
+			(at 3.5 2 0)
 			(layer "F.SilkS")
 			(effects
@@
 		(tags "C Disc series Radial pin pitch 5.00mm diameter 6mm width 2.5mm Capacitor")
 		(property "Reference" "C3"
-			(at 2.5 -2.5 90)
+			(at 2.5 -2.5 180)
 			(layer "F.SilkS")
 			(effects
@@
 	(footprint "Connector_PinHeader_2.54mm:PinHeader_1x06_P2.54mm_Vertical"
 		(layer "F.Cu")
-		(at 114 119.5 90)
+		(at 114 118.5 90)
 		(descr "Through hole straight pin header, 1x06, 2.54mm pitch, single row")
 		(tags "Through hole pin header THT 1x06 2.54mm single row")
@@
 		(tags "tact sw push 6mm")
 		(property "Reference" "SW1"
-			(at 3.25 7 0)
+			(at 5.5 -2.5 0)
 			(layer "F.SilkS")
 			(effects
@@
 		(tags "Through hole pin header THT 1x05 2.54mm single row")
 		(property "Reference" "J1"
-			(at 0 -2.38 0)
+			(at 0 -3 0)
 			(layer "F.SilkS")
 			(effects
@@
 		(tags "THT Terminal Block TE 282834-2 pitch 2.54mm size 5.54x6.5mm drill 1.1mm pad 2.1mm")
 		(property "Reference" "J5"
-			(at 1.27 -4.37 0)
+			(at 5.54 -3 0)
 			(layer "F.SilkS")
 			(effects
@@
 		(tags "C Disc series Radial pin pitch 5.00mm diameter 6mm width 2.5mm Capacitor")
 		(property "Reference" "C2"
-			(at 2.5 -2.5 90)
+			(at 7 0 180)
 			(layer "F.SilkS")
 			(effects
@@
 		)
 	)
+	(gr_rect
+		(start 104 70)
+		(end 140.5 121)
+		(stroke
+			(width 0.05)
+			(type default)
+		)
+		(fill no)
+		(layer "Edge.Cuts")
+	)
 	(embedded_fonts no)

Commit message: 20251228
Routing:
- net GND: track 0.00 -> 32.0 mm
- net Net-(U1-PC6): track 0.00 -> 21.8 mm
- net PB5: track 0.00 -> 14.6 mm
- net Net-(U1-PB6): track 0.00 -> 14.6 mm
- net PD7: track 0.00 -> 13.8 mm
- net TX: track 0.00 -> 13.8 mm
- net RX: track 0.00 -> 13.3 mm
- net PB4: track 0.00 -> 9.24 mm
- net PB2: track 0.00 -> 9.24 mm
- net PB3: track 0.00 -> 9.24 mm
- net PB1: track 0.00 -> 9.24 mm
- net PC5: track 0.00 -> 8.46 mm
- net PC3: track 0.00 -> 8.46 mm
- net PC1: track 0.00 -> 8.46 mm
- net PC4: track 0.00 -> 8.46 mm
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
Commit message: 20251229
Routing:
- net GND: track 32.0 -> 106.1 mm, vias 0 -> 3
- net +5V: track 4.62 -> 72.0 mm
- net DTR: track 0.00 -> 22.4 mm
- net PD4: track 0.00 -> 19.3 mm
- net PD3: track 0.00 -> 19.3 mm
- net PD2: track 0.00 -> 18.7 mm
- net PB0: track 0.00 -> 17.9 mm
- net PD6: track 0.00 -> 13.8 mm
- net PD5: track 0.00 -> 13.8 mm
- net PC0: track 0.00 -> 8.46 mm
- net Net-(U1-PB7): track 6.97 -> 12.2 mm

Commit message: 20251229
Connections:
- net Net-(U1-PC6) renamed RESET
Changed lines of the file:
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@@
 	(net 3 "+5V")
 	(net 4 "DTR")
-	(net 5 "Net-(U1-PC6)")
+	(net 5 "RESET")
 	(net 6 "Net-(U1-PB7)")
 	(net 7 "Net-(U1-PB6)")
@@
 			(layers "*.Cu" "*.Mask")
 			(remove_unused_layers no)
-			(net 5 "Net-(U1-PC6)")
+			(net 5 "RESET")
 			(pintype "passive")
 		)
@@
 			(remove_unused_layers no)
 			(roundrect_rratio 0.15625)
-			(net 5 "Net-(U1-PC6)")
+			(net 5 "RESET")
 			(pinfunction "PC6")
 			(pintype "bidirectional")
@@
 			(layers "*.Cu" "*.Mask")
 			(remove_unused_layers no)
-			(net 5 "Net-(U1-PC6)")
+			(net 5 "RESET")
 			(pintype "passive")
 		)
@@
 			(layers "*.Cu" "*.Mask")
 			(remove_unused_layers no)
-			(net 5 "Net-(U1-PC6)")
+			(net 5 "RESET")
 			(pinfunction "2")
 			(pintype "passive")
@@
 			(layers "*.Cu" "*.Mask")
 			(remove_unused_layers no)
-			(net 5 "Net-(U1-PC6)")
+			(net 5 "RESET")
 			(pinfunction "2")
 			(pintype "passive")

Commit message: 20260103
Connections:
- J2 pad 1: PD0 -> RX
- J2 pad 2: PD1 -> TX
Routing:
- net RX: track 13.3 -> 26.7 mm
- net TX: track 13.8 -> 26.3 mm
- added copper zone on F.Cu, net +5V
- added copper zone on B.Cu, net GND
Other:
- board size 36.5 x 51 mm -> 39.2 x 55 mm
- board text added: "+5V(DC,MAX)"
- board text added: "5V"
- board text added: "<-5V->"
- board text added: "<-GND->"
- board text added: "A0"
- board text added: "A1"
- board text added: "A2"
- board text added: "A3"
- board text added: "A4"
- board text added: "A5"
- board text added: "D10"
- board text added: "D11"
- board text added: "D12"
- board text added: "D13"
- board text added: "D2"
- board text added: "D3"
- board text added: "D4"
- board text added: "D5"
- board text added: "D6"
- board text added: "D7"
- board text added: "D8"
- board text added: "D9"
- board text added: "DTR"
- board text added: "GND"
- board text added: "RESET"
- board text added: "RX"
- board text added: "TX"
