File: Projects/Tutorial03-ESP32-IoT-4-layer-PCB/Tutorial03-ESP32-IoT-4-layer-PCB.kicad_sch (KiCad schematic)
At the start: 0 parts

Commit message: 20260131
Other:
- title: (none) -> ESP32 Sensor Board Root
Changed lines of the file:
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@@
 	(generator_version "9.0")
 	(paper "A4")
+	(title_block
+		(title "ESP32 Sensor Board Root")
+	)
 	(sheet_instances
 		(path "/"

Commit message: 20260131
Parts:
- added J1: SS-52400-002, SS-52400-002:BELFUSE_SS-52400-002, symbol SS-52400-002:SS-52400-002
- added J2: B2B-PH-SM4-TB, B2B-PH-SM4-TB:JST_B2B-PH-SM4-TB, symbol B2B-PH-SM4-TB:B2B-PH-SM4-TB
- added U1: MCP73871-2CAI_ML, MCP73871-2CAI_ML:QFN50P400X400X100-21N, symbol MCP73871-2CAI_ML:MCP73871-2CAI_ML
- added VR1: LM1117MPX-3.3, LM1117MPX-3.3:VREG_LM1117MPX-3.3, symbol LM1117MPX-3.3:LM1117MPX-3.3
Connections:
- new net: J1.G1 (GND/SHIELD), J1.G2 (GND/SHIELD), J1.G3 (GND/SHIELD), J1.G4 (GND/SHIELD), J1.S1 (GND/SHIELD), J1.S2 (GND/SHIELD), J1.S3 (GND/SHIELD), J1.S4 (GND/SHIELD)
- new net: U1.1 (OUT), U1.20 (OUT)
- new net: U1.10 (VSS), U1.11 (VSS), U1.21 (VSS)
- new net: U1.14 (VBAT), U1.15 (VBAT)
- new net: U1.18 (IN), U1.19 (IN)

Commit message: 20260131
Parts:
- removed U1: MCP73871-2CAI_ML, MCP73871-2CAI_ML:QFN50P400X400X100-21N, symbol MCP73871-2CAI_ML:MCP73871-2CAI_ML
- added LED1 (RED): LTST-C170KRKT, LEDC2012X120N, symbol LTST-C170KRKT:LTST-C170KRKT
- added LED2 (GREEN): LTST-C170GKT, LEDC2012X120N, symbol LTST-C170GKT:LTST-C170GKT
- added LED3 (BLUE): LTST-C170TBKT, LEDC2012X120N, symbol LTST-C170TBKT:LTST-C170TBKT
- added R1, R2: 10K, symbol Device:R
- added R3, R4: 5K1, symbol Device:R
- added R5: 2K, symbol Device:R
- added R6: 20K, symbol Device:R
- added R7, R8, R9: 470, symbol Device:R
- added U1: MCP73871, Package_DFN_QFN:QFN-20-1EP_4x4mm_P0.5mm_EP2.5x2.5mm, symbol Battery_Management:MCP73871
Connections:
- net at J1.A5 (CC1): now also R4.1
- net at J1.B5 (CC2): now also R3.1
- new net: LED3 (BLUE).1 (K), R9.2
- new net: R7.1, U1.7 (STAT2)
- new net: LED1 (RED).1 (K), R7.2
- new net: R1.1, U1.9 (~{TE})
- new net: LED2 (GREEN).1 (K), R8.2
- new net: R8.1, U1.8 (STAT1/~{LBO})
- new net: R6.1, U1.12 (PROG3)
- new net: R9.1, U1.6 (~{PG})
- new net: U1.1 (OUT), U1.20 (OUT)
- new net: U1.10 (V_{SS}), U1.11 (V_{SS}), U1.21 (V_{SS})
- new net: R5.1, U1.13 (PROG1)
- new net: U1.14 (V_{BAT}), U1.15 (V_{BAT})
- new net: U1.18 (IN), U1.19 (IN)
- new net: R2.1, U1.5 (THERM)
- new net GND: LED1 (RED).2 (A), LED2 (GREEN).2 (A), LED3 (BLUE).2 (A), R1.2, R2.2, R5.2, R6.2

Commit message: 20260205
Connections:
- net GND: now also J1.A1 (GNDA1), J1.A12 (GNDA2), J1.B1 (GNDB1), J1.B12 (GNDB2), J1.G1 (GND/SHIELD), J1.G2 (GND/SHIELD), J1.G3 (GND/SHIELD), J1.G4 (GND/SHIELD), J1.S1 (GND/SHIELD), J1.S2 (GND/SHIELD), J1.S3 (GND/SHIELD), J1.S4 (GND/SHIELD), R3.2, R4.2; no longer LED1 (RED).2 (A), LED2 (GREEN).2 (A), LED3 (BLUE).2 (A)
Other:
- moved on the sheet: R3

Commit message: 20260205
Parts:
- added F1: 0ZCH0110AF2E, FUSC3226X100N, symbol 0ZCH0110AF2E:0ZCH0110AF2E
Changed lines of the file:
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@@
+	)
+	(symbol
+		(lib_id "0ZCH0110AF2E:0ZCH0110AF2E")
+		(at 105.41 69.85 0)
+		(unit 1)
+		(exclude_from_sim no)
+		(in_bom yes)
+		(on_board yes)
+		(dnp no)
+		(fields_autoplaced yes)
+		(property "Reference" "F1"
+			(at 114.3 63.5 0)
+			(effects
+				(font
+					(size 1.27 1.27)
+				)
+			)
+		)
+		(property "Value" "0ZCH0110AF2E"
+			(at 114.3 66.04 0)
+			(effects
+				(font
+					(size 1.27 1.27)
+				)
+			)
+		)
+		(property "Footprint" "FUSC3226X100N"
+			(at 119.38 166.04 0)
+			(effects
+				(font
+					(size 1.27 1.27)
+				)
+				(justify left top)
+				(hide yes)
+			)
+		)
+		(property "Datasheet" "https://www.belfuse.com/resources/datasheets/circuitprotection/ds-cp-0zch-series.pdf"
+			(at 119.38 266.04 0)
+			(effects
+				(font
+					(size 1.27 1.27)
+				)
+				(justify left top)
+				(hide yes)
+			)
+		)
+		(property "Description" "1210 SMT PPTC | 1.10 Ih | 16V"
+			(at 105.41 69.85 0)
+			(effects
+				(font
+					(size 1.27 1.27)
+				)
+				(hide yes)
+			)
+		)
+		(property "Height" "1"
+			(at 119.38 466.04 0)
+			(effects
+				(font
+					(size 1.27 1.27)
+				)
+				(justify left top)
+				(hide yes)
+			)
+		)
+		(property "Manufacturer_Name" "Bel Circuit Protection"
+			(at 119.38 566.04 0)
+			(effects
+				(font
+					(size 1.27 1.27)
+				)
+				(justify left top)
+				(hide yes)
+			)
+		)
+		(property "Manufacturer_Part_Number" "0ZCH0110AF2E"
+			(at 119.38 666.04 0)
+			(effects
+				(font
+					(size 1.27 1.27)
+				)
+				(justify left top)
+				(hide yes)
+			)
+		)
+		(property "Mouser Part Number" ""
+			(at 119.38 766.04 0)
+			(effects
+				(font
+					(size 1.27 1.27)
+				)
+				(justify left top)
+				(hide yes)
+			)
+		)
+		(property "Mouser Price/Stock" ""
+			(at 119.38 866.04 0)
+			(effects
+				(font
+					(size 1.27 1.27)
+				)
+				(justify left top)
+				(hide yes)
+			)
+		)
+		(property "Arrow Part Number" ""
+			(at 119.38 966.04 0)
+			(effects
+				(font
+					(size 1.27 1.27)
+				)
+				(justify left top)
+				(hide yes)
+			)
+		)
+		(property "Arrow Price/Stock" ""
+			(at 119.38 1066.04 0)
+			(effects
+				(font
+					(size 1.27 1.27)
+				)
+				(justify left top)
+				(hide yes)
+			)
+		)
+		(pin "2"
+		)
+		(pin "1"
+		)
+		(instances
+			(project ""
+				(path "/49253bfd-5dbd-467b-ba3c-7c0c524516c8"
+					(reference "F1")
+					(unit 1)
+				)
+			)
+		)
 	)
 	(symbol

Commit message: 20260207
Parts:
- added C1: 0.1u, symbol Device:C
- added C2: C, symbol Device:C
Connections:
- net GND: now also C1.2
- net at J1.B4 (VBUSB1): now also F1.1, C1.1
- no-connect marks 0 -> 10
Other:
- moved on the sheet: F1, J1, LED1 (RED), LED2 (GREEN), LED3 (BLUE), R1, R2, R3, R4, R5, R6, R7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

Commit message: 20260207
Connections:
- net +5V_USB: now reaches LED3 (BLUE).2 (A)
- net +5V_USB: now also F1.2, LED1 (RED).2 (A), LED2 (GREEN).2 (A)
- net VUSB: now reaches J1.A4 (VBUSA1)
- net VUSB: now also C1.1, F1.1, J1.A9 (VBUSA2), J1.B4 (VBUSB1), J1.B9 (VBUSB2)
- net USB_DP: now reaches J1.A6 (DP1)
- net USB_DP: now also J1.B6 (DP2)
- net USB_DN: now reaches J1.A7 (DN1)
- net USB_DN: now also J1.B7 (DN2)
Other:
- note added: "USB-C CONNECTOR"
- moved on the sheet: C1, C2, F1, J1, R3, R4

Commit message: 20260214
Parts:
- C6: renamed from C2; value C -> 1u
Connections:
- net +5V_USB: now also C6.1, U1.17 (CE), U1.18 (IN), U1.19 (IN), U1.2 (VPCC), U1.4 (PROG2)
- net GND: now also C6.2, U1.10 (V_{SS}), U1.11 (V_{SS}), U1.21 (V_{SS})
- net +5V: now reaches U1.1 (OUT), U1.20 (OUT)
- net VBAT: now reaches U1.14 (V_{BAT}), U1.15 (V_{BAT})
- net VBAT: now also U1.16 (V_{BAT_SENSE})
Other:
- note added: "LiPo (Lithium Polymer) battery charger"
- moved on the sheet: C6, LED1 (RED), LED2 (GREEN), LED3 (BLUE), R1, R2, R5, R6, R7, R8, R9, U1
