File: Projects/Tutorial03-ESP32-IoT-4-layer-PCB/Tutorial03-ESP32-IoT-4-layer-PCB.kicad_sch (KiCad schematic)
At the start: 19 parts, among them J1 SS-52400-002, J2 B2B-PH-SM4-TB, U1 MCP73871

Commit message: 20260214
Parts:
- added C2, C5: 0.1u, symbol Device:C
- added C3, C4: 10u, symbol Device:C_Polarized
- added LED1 (RED)1: LTST-C170KRKT, LEDC2012X120N, symbol LTST-C170KRKT:LTST-C170KRKT
- added R10: 470, symbol Device:R
Connections:
- net +5V: now also VR1.3 (VIN), C2.1, C3.1
- net GND: now also J2.1, VR1.1 (GND), C2.2, C3.2, C4.2, C5.2, R10.1
- net VBAT: now also J2.2
- net +3.3V: now reaches VR1.2 (VOUT_2)
- net +3.3V: now also VR1.4 (VOUT_4), C4.1, C5.1, LED1 (RED)1.2 (A)
- new net: LED1 (RED)1.1 (K), R10.2
Other:
- note added: "Battery JST Connector"
- note added: "LDO (Low Dropout) Voltage Regulator"
- note added: "Power INdicator LED"
- moved on the sheet: J2, VR1

Commit message: 20260220
Connections:
- net at LED3 (BLUE).1 (K): now also R7.2; no longer R9.2
- net at LED1 (RED).1 (K): now also R9.2; no longer R7.2
- net CHARGING: now reaches R9.1, U1.6 (~{PG})
Other:
- added sheet ESP-32-C3-02 (esp-32-c3-02.kicad_sch)
- moved on the sheet: LED1 (RED), LED3 (BLUE)

Commit message: 20260221
Connections:
- net VUSB renamed VBUS
Other:
- sheet ESP-32-C3-02 ports: added USB_DN, USB_DP, VBUS; removed none
Changed lines of the file:
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@@
 	(wire
 		(pts
+			(xy 134.62 153.67) (xy 137.16 153.67)
+		)
+		(stroke
+			(width 0)
+			(type default)
+		)
+	)
+	(wire
+		(pts
 			(xy 123.19 107.95) (xy 111.76 107.95)
 		)
@@
 	(wire
 		(pts
+			(xy 134.62 149.86) (xy 137.16 149.86)
+		)
+		(stroke
+			(width 0)
+			(type default)
+		)
+	)
+	(wire
+		(pts
 			(xy 266.7 68.58) (xy 266.7 71.12)
 		)
@@
 	(wire
 		(pts
+			(xy 134.62 147.32) (xy 137.16 147.32)
+		)
+		(stroke
+			(width 0)
+			(type default)
+		)
+	)
+	(wire
+		(pts
 			(xy 52.07 105.41) (xy 52.07 107.95)
 		)
@@
 		)
 	)
-	(label "VUSB"
+	(label "VBUS"
 		(at 87.63 50.8 0)
 		(effects
@@
 		)
 	)
-	(label "VUSB"
+	(label "VBUS"
 		(at 44.45 38.1 180)
 		(effects
@@
 		)
 	)
+	(label "VBUS"
+		(at 137.16 153.67 0)
+		(effects
+			(font
+				(size 1.27 1.27)
+			)
+			(justify left bottom)
+		)
+	)
 	(label "USB_DP"
 		(at 44.45 43.18 180)
@@
 		)
 	)
-	(label "VUSB"
+	(label "VBUS"
 		(at 92.71 38.1 180)
 		(effects
@@
 		)
 	)
-	(label "VUSB"
+	(label "USB_DN"
+		(at 137.16 149.86 0)
+		(effects
+			(font
+				(size 1.27 1.27)
+			)
+			(justify left bottom)
+		)
+	)
+	(label "VBUS"
 		(at 44.45 50.8 180)
 		(effects
@@
 		)
 	)
+	(label "USB_DP"
+		(at 137.16 147.32 0)
+		(effects
+			(font
+				(size 1.27 1.27)
+			)
+			(justify left bottom)
+		)
+	)
 	(label "VBAT"
 		(at 205.74 53.34 180)
@@
 	)
 	(sheet
-		(at 80.01 144.78)
+		(at 76.2 144.78)
 		(size 58.42 24.13)
 		(exclude_from_sim no)
@@
 		)
 		(property "Sheetname" "ESP-32-C3-02"
-			(at 80.01 144.0684 0)
+			(at 76.2 144.0684 0)
 			(effects
 				(font
@@
 		)
 		(property "Sheetfile" "esp-32-c3-02.kicad_sch"
-			(at 80.01 169.4946 0)
+			(at 76.2 169.4946 0)
 			(effects
 				(font
@@
 			)
 		)
+		(pin "USB_DN" input
+			(at 134.62 149.86 0)
+			(effects
+				(font
+					(size 1.27 1.27)
+				)
+				(justify right)
+			)
+		)
+		(pin "USB_DP" input
+			(at 134.62 147.32 0)
+			(effects
+				(font
+					(size 1.27 1.27)
+				)
+				(justify right)
+			)
+		)
+		(pin "VBUS" input
+			(at 134.62 153.67 0)
+			(effects
+				(font
+					(size 1.27 1.27)
+				)
+				(justify right)
+			)
+		)

Commit message: 20260301
Parts:
- LED1-RED: renamed from LED1 (RED)
- LED2-GREEN: renamed from LED2 (GREEN)
- LED3-BLUE: renamed from LED3 (BLUE)
Changed lines of the file:
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@@
 		(on_board yes)
 		(dnp no)
-		(property "Reference" "LED3 (BLUE)"
+		(property "Reference" "LED3-BLUE"
 			(at 163.068 61.722 0)
 			(effects
@@
 			(project ""
 				(path "/49253bfd-5dbd-467b-ba3c-7c0c524516c8"
-					(reference "LED3 (BLUE)")
+					(reference "LED3-BLUE")
 					(unit 1)
 				)
@@
 		(on_board yes)
 		(dnp no)
-		(property "Reference" "LED2 (GREEN)"
+		(property "Reference" "LED2-GREEN"
 			(at 176.784 62.23 0)
 			(effects
@@
 			(project ""
 				(path "/49253bfd-5dbd-467b-ba3c-7c0c524516c8"
-					(reference "LED2 (GREEN)")
+					(reference "LED2-GREEN")
 					(unit 1)
 				)
@@
 		(on_board yes)
 		(dnp no)
-		(property "Reference" "LED1 (RED)"
+		(property "Reference" "LED1-RED"
 			(at 190.5 60.452 0)
 			(effects
@@
 			(project ""
 				(path "/49253bfd-5dbd-467b-ba3c-7c0c524516c8"
-					(reference "LED1 (RED)")
-					(unit 1)
-				)
+					(reference "LED1-RED")
+					(unit 1)
+				)

Commit message: 20260425
Parts:
- renumbered LED1-RED to LED1-RED1, LED2-GREEN to LED2-GREEN1, LED3-BLUE to LED3-BLUE1
Changed lines of the file:
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@@
 		)
 		(instances
-			(project ""
+			(project "Tutorial03-ESP32-IoT-4-layer-PCB"
 				(path "/49253bfd-5dbd-467b-ba3c-7c0c524516c8"
 					(reference "VR1")
@@
 		(on_board yes)
 		(dnp no)
-		(property "Reference" "LED3-BLUE"
+		(property "Reference" "LED3-BLUE1"
 			(at 163.068 61.722 0)
 			(effects
@@
 		)
 		(instances
-			(project ""
+			(project "Tutorial03-ESP32-IoT-4-layer-PCB"
 				(path "/49253bfd-5dbd-467b-ba3c-7c0c524516c8"
-					(reference "LED3-BLUE")
+					(reference "LED3-BLUE1")
 					(unit 1)
 				)
@@
 		)
 		(instances
-			(project ""
+			(project "Tutorial03-ESP32-IoT-4-layer-PCB"
 				(path "/49253bfd-5dbd-467b-ba3c-7c0c524516c8"
 					(reference "R7")
@@
 		)
 		(instances
-			(project ""
+			(project "Tutorial03-ESP32-IoT-4-layer-PCB"
 				(path "/49253bfd-5dbd-467b-ba3c-7c0c524516c8"
 					(reference "J1")
@@
 		)
 		(instances
-			(project ""
+			(project "Tutorial03-ESP32-IoT-4-layer-PCB"
 				(path "/49253bfd-5dbd-467b-ba3c-7c0c524516c8"
 					(reference "#PWR01")
@@
 		)
 		(instances
-			(project ""
+			(project "Tutorial03-ESP32-IoT-4-layer-PCB"
 				(path "/49253bfd-5dbd-467b-ba3c-7c0c524516c8"
 					(reference "R1")
@@
 		)
 		(instances
-			(project ""
+			(project "Tutorial03-ESP32-IoT-4-layer-PCB"
 				(path "/49253bfd-5dbd-467b-ba3c-7c0c524516c8"
 					(reference "C1")
@@
 		(on_board yes)
 		(dnp no)
-		(property "Reference" "LED2-GREEN"
+		(property "Reference" "LED2-GREEN1"
 			(at 176.784 62.23 0)
 			(effects
@@
 		)
 		(instances
-			(project ""
+			(project "Tutorial03-ESP32-IoT-4-layer-PCB"
 				(path "/49253bfd-5dbd-467b-ba3c-7c0c524516c8"
-					(reference "LED2-GREEN")
+					(reference "LED2-GREEN1")
 					(unit 1)
 				)
@@
 		)
 		(instances
-			(project ""
+			(project "Tutorial03-ESP32-IoT-4-layer-PCB"
 				(path "/49253bfd-5dbd-467b-ba3c-7c0c524516c8"
 					(reference "J2")
@@
 		)
 		(instances
-			(project ""
+			(project "Tutorial03-ESP32-IoT-4-layer-PCB"
 				(path "/49253bfd-5dbd-467b-ba3c-7c0c524516c8"
 					(reference "R3")
@@
 		)
 		(instances
-			(project ""
+			(project "Tutorial03-ESP32-IoT-4-layer-PCB"
 				(path "/49253bfd-5dbd-467b-ba3c-7c0c524516c8"
 					(reference "C3")
@@
 		)
 		(instances
-			(project ""
+			(project "Tutorial03-ESP32-IoT-4-layer-PCB"
 				(path "/49253bfd-5dbd-467b-ba3c-7c0c524516c8"
 					(reference "#PWR011")
@@
 		)
 		(instances
-			(project ""
+			(project "Tutorial03-ESP32-IoT-4-layer-PCB"
 				(path "/49253bfd-5dbd-467b-ba3c-7c0c524516c8"
 					(reference "C6")
@@
 		)
 		(instances
-			(project ""
+			(project "Tutorial03-ESP32-IoT-4-layer-PCB"
 				(path "/49253bfd-5dbd-467b-ba3c-7c0c524516c8"
 					(reference "#PWR013")
@@
 		)
 		(instances
-			(project ""
+			(project "Tutorial03-ESP32-IoT-4-layer-PCB"
 				(path "/49253bfd-5dbd-467b-ba3c-7c0c524516c8"
 					(reference "U1")
@@
 		(on_board yes)
 		(dnp no)
-		(property "Reference" "LED1-RED"
+		(property "Reference" "LED1-RED1"
 			(at 190.5 60.452 0)
 			(effects
@@
 		)
 		(instances
-			(project ""
+			(project "Tutorial03-ESP32-IoT-4-layer-PCB"
 				(path "/49253bfd-5dbd-467b-ba3c-7c0c524516c8"
-					(reference "LED1-RED")
+					(reference "LED1-RED1")
 					(unit 1)
 				)
@@
 		)
 		(instances
-			(project ""
+			(project "Tutorial03-ESP32-IoT-4-layer-PCB"
 				(path "/49253bfd-5dbd-467b-ba3c-7c0c524516c8"
 					(reference "F1")
@@
 		)
 		(instances
-			(project ""
+			(project "Tutorial03-ESP32-IoT-4-layer-PCB"
 				(path "/49253bfd-5dbd-467b-ba3c-7c0c524516c8"
 					(reference "#FLG01")

Commit message: 20260425
Parts:
- C1, C2, C5, C6: footprint (none) -> Capacitor_SMD:C_0805_2012Metric
- C3, C4: footprint (none) -> ESP32 Project Footprints:T491A
- F1: footprint FUSC3226X100N -> ESP32 Project Footprints:FUSC3226X100N
- J1: footprint SS-52400-002:BELFUSE_SS-52400-002 -> ESP32 Project Footprints:BELFUSE_SS-52400-002
- J2: footprint B2B-PH-SM4-TB:JST_B2B-PH-SM4-TB -> ESP32 Project Footprints:JST_B2B-PH-SM4-TB
- LED1 (RED)1: footprint LEDC2012X120N -> ESP32 Project Footprints:LEDC2012X120N
- LED1-RED1, LED2-GREEN1, LED3-BLUE1: footprint LEDC2012X120N -> ESP32 Project Footprints:LEDC2012X120N
- R1, R10, R2, R3, R4, R5, R6, R7, R8, R9: footprint (none) -> Resistor_SMD:R_0805_2012Metric
Changed lines of the file:
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@@
 			)
 		)
-		(property "Footprint" ""
+		(property "Footprint" "Resistor_SMD:R_0805_2012Metric"
 			(at 194.31 107.442 90)
 			(effects
@@
 			)
 		)
-		(property "Footprint" "LEDC2012X120N"
+		(property "Footprint" "ESP32 Project Footprints:LEDC2012X120N"
 			(at 73.99 69.85 0)
 			(effects
@@
 			)
 		)
-		(property "Footprint" ""
+		(property "Footprint" "Resistor_SMD:R_0805_2012Metric"
 			(at 165.862 49.53 90)
 			(effects
@@
 			)
 		)
-		(property "Footprint" "SS-52400-002:BELFUSE_SS-52400-002"
+		(property "Footprint" "ESP32 Project Footprints:BELFUSE_SS-52400-002"
 			(at 66.04 45.72 0)
 			(effects
@@
 			)
 		)
-		(property "Footprint" ""
+		(property "Footprint" "ESP32 Project Footprints:T491A"
 			(at 110.7948 118.11 0)
 			(effects
@@
 			)
 		)
-		(property "Footprint" ""
+		(property "Footprint" "Capacitor_SMD:C_0805_2012Metric"
 			(at 53.0352 115.57 0)
 			(effects
@@
 			)
 		)
-		(property "Footprint" ""
+		(property "Footprint" "Resistor_SMD:R_0805_2012Metric"
 			(at 259.08 39.878 90)
 			(effects
@@
 			)
 		)
-		(property "Footprint" ""
+		(property "Footprint" "Capacitor_SMD:C_0805_2012Metric"
 			(at 113.9952 54.61 0)
 			(effects
@@
 			)
 		)
-		(property "Footprint" "LEDC2012X120N"
+		(property "Footprint" "ESP32 Project Footprints:LEDC2012X120N"
 			(at 87.96 69.85 0)
 			(effects
@@
 			)
 		)
-		(property "Footprint" "B2B-PH-SM4-TB:JST_B2B-PH-SM4-TB"
+		(property "Footprint" "ESP32 Project Footprints:JST_B2B-PH-SM4-TB"
 			(at 44.45 153.67 0)
 			(effects
@@
 			)
 		)
-		(property "Footprint" ""
+		(property "Footprint" "Resistor_SMD:R_0805_2012Metric"
 			(at 99.822 50.8 90)
 			(effects
@@
 			)
 		)
-		(property "Footprint" ""
+		(property "Footprint" "ESP32 Project Footprints:T491A"
 			(at 65.7352 115.57 0)
 			(effects
@@
 			)
 		)
-		(property "Footprint" ""
+		(property "Footprint" "Capacitor_SMD:C_0805_2012Metric"
 			(at 228.2952 83.82 0)
 			(effects
@@
 			)
 		)
-		(property "Footprint" ""
+		(property "Footprint" "Resistor_SMD:R_0805_2012Metric"
 			(at 179.832 49.53 90)
 			(effects
@@
 			)
 		)
-		(property "Footprint" ""
+		(property "Footprint" "Resistor_SMD:R_0805_2012Metric"
 			(at 32.512 59.69 90)
 			(effects
@@
 			)
 		)
-		(property "Footprint" ""
+		(property "Footprint" "Resistor_SMD:R_0805_2012Metric"
 			(at 264.922 64.77 90)
 			(effects
@@
 			)
 		)
-		(property "Footprint" ""
+		(property "Footprint" "Resistor_SMD:R_0805_2012Metric"
 			(at 193.802 48.26 90)
 			(effects
@@
 			)
 		)
-		(property "Footprint" "LEDC2012X120N"
+		(property "Footprint" "ESP32 Project Footprints:LEDC2012X120N"
 			(at 175.26 15.57 0)
 			(effects
@@
 			)
 		)
-		(property "Footprint" ""
+		(property "Footprint" "Resistor_SMD:R_0805_2012Metric"
 			(at 259.08 44.958 90)
 			(effects
@@
 			)
 		)
-		(property "Footprint" "LEDC2012X120N"
+		(property "Footprint" "ESP32 Project Footprints:LEDC2012X120N"
 			(at 101.93 69.85 0)
 			(effects
@@
 			)
 		)
-		(property "Footprint" ""
+		(property "Footprint" "Resistor_SMD:R_0805_2012Metric"
 			(at 256.032 64.77 90)
 			(effects
@@
 			)
 		)
-		(property "Footprint" "FUSC3226X100N"
+		(property "Footprint" "ESP32 Project Footprints:FUSC3226X100N"
 			(at 133.35 134.29 0)
 			(effects
@@
 			)
 		)
-		(property "Footprint" ""
+		(property "Footprint" "Capacitor_SMD:C_0805_2012Metric"
 			(at 122.2248 118.11 0)
 			(effects

Commit message: 20260425
Connections:
- net CHARGED: now also R8.1, U1.8 (STAT1/~{LBO})
- net GND: now also U1.3 (SEL)
- net POWER_CHARGING_GOOD: now also R7.1, U1.7 (STAT2)
