File: Projects/Tutorial03-ESP32-IoT-4-layer-PCB/Tutorial03-ESP32-IoT-4-layer-PCB.kicad_sch (KiCad schematic)
At the start: 25 parts, among them J1 SS-52400-002, J2 B2B-PH-SM4-TB, U1 MCP73871

Commit message: 20260516
Parts:
- VR1: footprint LM1117MPX-3.3:VREG_LM1117MPX-3.3 -> ESP32 Project Footprints:VREG_LM1117MPX-3.3
Changed lines of the file:
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@@
 			)
 		)
-		(property "Footprint" "LM1117MPX-3.3:VREG_LM1117MPX-3.3"
+		(property "Footprint" "ESP32 Project Footprints:VREG_LM1117MPX-3.3"
 			(at 87.63 107.95 0)
 			(effects
@@
 				)
 				(justify bottom)
-				(hide yes)
 			)
 		)

Commit message: 20260516
Parts:
- removed VR1: LM1117MPX-3.3, ESP32 Project Footprints:VREG_LM1117MPX-3.3, symbol LM1117MPX-3.3:LM1117MPX-3.3
- added VR1: LM1117MPX-3.3, ESP32 Project Footprints:VREG_LM1117MPX-3.3, symbol PRJ-LM1117MPX-3.3:LM1117MPX-3.3
Connections:
- net +3.3V: now also VR1.2 (VOUT_2), VR1.4 (VOUT_4)
- net +5V: now also VR1.3 (VIN)
- net GND: now also VR1.1 (GND)

Commit message: 20260516
Parts:
- removed VR1: LM1117MPX-3.3, ESP32 Project Footprints:VREG_LM1117MPX-3.3, symbol PRJ-LM1117MPX-3.3:LM1117MPX-3.3
- added VR1: LM1117MPX-3.3, ESP32 Project Footprints:VREG_LM1117MPX-3.3, symbol LM1117MPX-3.3:LM1117MPX-3.3
Connections:
- net +3.3V: now also VR1.2 (VOUT_2), VR1.4 (VOUT_4)
- net +5V: now also VR1.3 (VIN)
- net GND: now also VR1.1 (GND)

Commit message: 20260525
Parts:
- C3, C4: footprint ESP32 Project Footprints:T491A -> Project-Footprints:T491A
- F1: footprint ESP32 Project Footprints:FUSC3226X100N -> Project-Footprints:FUSC3226X100N
- J1: footprint ESP32 Project Footprints:BELFUSE_SS-52400-002 -> Project-Footprints:BELFUSE_SS-52400-002
- J2: footprint ESP32 Project Footprints:JST_B2B-PH-SM4-TB -> Project-Footprints:JST_B2B-PH-SM4-TB
- LED1-RED1, LED2-GREEN1, LED3-BLUE1: footprint ESP32 Project Footprints:LEDC2012X120N -> Project-Footprints:LEDC2012X120N
- LED2-RED1: renamed from LED1 (RED)1; footprint ESP32 Project Footprints:LEDC2012X120N -> Project-Footprints:LEDC2012X120N
- VR1: footprint ESP32 Project Footprints:VREG_LM1117MPX-3.3 -> Project-Footprints:VREG_LM1117MPX-3.3
Changed lines of the file:
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@@
 			)
 		)
-		(property "Footprint" "ESP32 Project Footprints:LEDC2012X120N"
+		(property "Footprint" "Project-Footprints:LEDC2012X120N"
 			(at 73.99 69.85 0)
 			(effects
@@
 			)
 		)
-		(property "Footprint" "ESP32 Project Footprints:BELFUSE_SS-52400-002"
+		(property "Footprint" "Project-Footprints:BELFUSE_SS-52400-002"
 			(at 66.04 45.72 0)
 			(effects
@@
 			)
 		)
-		(property "Footprint" "ESP32 Project Footprints:T491A"
+		(property "Footprint" "Project-Footprints:T491A"
 			(at 110.7948 118.11 0)
 			(effects
@@
 			)
 		)
-		(property "Footprint" "ESP32 Project Footprints:LEDC2012X120N"
+		(property "Footprint" "Project-Footprints:LEDC2012X120N"
 			(at 87.96 69.85 0)
 			(effects
@@
 			)
 		)
-		(property "Footprint" "ESP32 Project Footprints:JST_B2B-PH-SM4-TB"
+		(property "Footprint" "Project-Footprints:JST_B2B-PH-SM4-TB"
 			(at 44.45 153.67 0)
 			(effects
@@
 			)
 		)
-		(property "Footprint" "ESP32 Project Footprints:VREG_LM1117MPX-3.3"
+		(property "Footprint" "Project-Footprints:VREG_LM1117MPX-3.3"
 			(at 86.36 107.95 0)
 			(effects
@@
 			)
 		)
-		(property "Footprint" "ESP32 Project Footprints:T491A"
+		(property "Footprint" "Project-Footprints:T491A"
 			(at 65.7352 115.57 0)
 			(effects
@@
 		(on_board yes)
 		(dnp no)
-		(property "Reference" "LED1 (RED)1"
+		(property "Reference" "LED2-RED1"
 			(at 184.658 104.14 0)
 			(effects
@@
 			)
 		)
-		(property "Footprint" "ESP32 Project Footprints:LEDC2012X120N"
+		(property "Footprint" "Project-Footprints:LEDC2012X120N"
 			(at 175.26 15.57 0)
 			(effects
@@
 			(project "Tutorial03-ESP32-IoT-4-layer-PCB"
 				(path "/49253bfd-5dbd-467b-ba3c-7c0c524516c8"
-					(reference "LED1 (RED)1")
+					(reference "LED2-RED1")
 					(unit 1)
 				)
@@
 			)
 		)
-		(property "Footprint" "ESP32 Project Footprints:LEDC2012X120N"
+		(property "Footprint" "Project-Footprints:LEDC2012X120N"
 			(at 101.93 69.85 0)
 			(effects
@@
 			)
 		)
-		(property "Footprint" "ESP32 Project Footprints:FUSC3226X100N"
+		(property "Footprint" "Project-Footprints:FUSC3226X100N"
 			(at 133.35 134.29 0)
 			(effects

Commit message: 20260620
Parts:
- renumbered LED1-RED1 to LED1R1, LED2-GREEN1 to LED2G1, LED3-BLUE1 to LED3B1
Changed lines of the file:
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@@
 		(on_board yes)
 		(dnp no)
-		(property "Reference" "LED3-BLUE1"
+		(property "Reference" "LED3B1"
 			(at 163.068 61.722 0)
 			(effects
@@
 			(project "Tutorial03-ESP32-IoT-4-layer-PCB"
 				(path "/49253bfd-5dbd-467b-ba3c-7c0c524516c8"
-					(reference "LED3-BLUE1")
+					(reference "LED3B1")
 					(unit 1)
 				)
@@
 		(on_board yes)
 		(dnp no)
-		(property "Reference" "LED2-GREEN1"
+		(property "Reference" "LED2G1"
 			(at 176.784 62.23 0)
 			(effects
@@
 			(project "Tutorial03-ESP32-IoT-4-layer-PCB"
 				(path "/49253bfd-5dbd-467b-ba3c-7c0c524516c8"
-					(reference "LED2-GREEN1")
+					(reference "LED2G1")
 					(unit 1)
 				)
@@
 		(on_board yes)
 		(dnp no)
-		(property "Reference" "LED1-RED1"
+		(property "Reference" "LED1R1"
 			(at 190.5 60.452 0)
 			(effects
@@
 			(project "Tutorial03-ESP32-IoT-4-layer-PCB"
 				(path "/49253bfd-5dbd-467b-ba3c-7c0c524516c8"
-					(reference "LED1-RED1")
-					(unit 1)
-				)
+					(reference "LED1R1")
+					(unit 1)
+				)

Commit message: 20260625
Parts:
- renumbered LED2-RED1 to LED2R1
Changed lines of the file:
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@@
 		(on_board yes)
 		(dnp no)
-		(property "Reference" "LED2-RED1"
+		(property "Reference" "LED2R1"
 			(at 184.658 104.14 0)
 			(effects
@@
 			(project "Tutorial03-ESP32-IoT-4-layer-PCB"
 				(path "/49253bfd-5dbd-467b-ba3c-7c0c524516c8"
-					(reference "LED2-RED1")
+					(reference "LED2R1")
 					(unit 1)
 				)
