File: Projects/Tutorial03-ESP32-IoT-4-layer-PCB/esp-32-c3-02.kicad_sch (KiCad schematic)
At the start: 0 parts

Commit message: 20260221
Parts:
- added J?: GSD090012SEU, GSD090012SEU:AMPHENOL_GSD090012SEU, symbol GSD090012SEU:GSD090012SEU
- added U2: USBLC6-2SC6, Package_TO_SOT_SMD:SOT-23-6, symbol Power_Protection:USBLC6-2SC6
- added U?: W25Q32JVSSIQ, W25Q32JVSSIQ:SOIC127P790X216-8N, symbol W25Q32JVSSIQ:W25Q32JVSSIQ
- added U?: ESP32-C3-WROOM-02-H4, ESP32-C3-WROOM-02-H4:MODULE_ESP32-C3-WROOM-02-H4, symbol ESP32-C3-WROOM-02-H4:ESP32-C3-WROOM-02-H4
- added U?: CP2102N-Axx-xQFN20, Package_DFN_QFN:SiliconLabs_QFN-20-1EP_3x3mm_P0.5mm, symbol Interface_USB:CP2102N-Axx-xQFN20
Connections:
- new net: U?.19 (GND), U?.20 (GND), U?.21 (GND), U?.22 (GND), U?.23 (GND), U?.24 (GND), U?.25 (GND), U?.26 (GND), U?.27 (GND), U?.28 (GND), U?.29 (GND), U?.30 (GND), U?.31 (GND), U?.32 (GND), U?.33 (GND), U?.34 (GND), U?.35 (GND), U?.36 (GND), U?.37 (GND), U?.38 (GND), U?.39 (GND), U?.9 (GND)
- new net: U?.12 (GND), U?.21 (GND), U?.3 (GND)
- new net: J?.G1 (SHIELD_GND), J?.G2 (SHIELD_GND), J?.G3 (SHIELD_GND), J?.G4 (SHIELD_GND)

Commit message: 20260221
Parts:
- added R12: 22K1, symbol Device:R
- added R13: 47K5, symbol Device:R
- gave numbers to parts that had none: 4
- renumbered U2 to U5
Connections:
- net at U5.1 (I/O1): now also U4.5 (D-)
- net GND: now reaches U5.2 (GND)
- net GND: now also R13.2
- net at U5.3 (I/O2): now also U4.4 (D+)
- net USB_DP: now reaches U5.4 (I/O2)
- net USB_DN: now reaches U5.6 (I/O1)
- net at U4.8 (VBUS): now also R12.2, R13.1
- new net VBUS: R12.1
Other:
- moved on the sheet: U5

Commit message: 20260221
Parts:
- added C11: 1u, symbol Device:C
- added C7: C, symbol Device:C
- added C8: C_Polarized, symbol Device:C_Polarized
- added R11: 1k, symbol Device:R
Connections:
- net GND: now also U4.12 (GND), U4.21 (GND), U4.3 (GND), C11.2
- net VBUS: now also U5.5 (VBUS)
- net at R12.2, R13.1, U4.8 (VBUS): now also C11.1
- net USB_D-: now reaches U4.5 (D-), U5.1 (I/O1)
- net USB_D+: now reaches U4.4 (D+), U5.3 (I/O2)
- net at U4.6 (VDD): now also U4.7 (VREGIN), R11.1
- net at U4.9 (~{RST}): now also R11.2
Other:
- moved on the sheet: R12, R13

Commit message: 20260301
Parts:
- added LED5-GREEN: LTST-C170GKT, LEDC2012X120N, symbol LTST-C170GKT:LTST-C170GKT
- added LED6-RED: LTST-C170KRKT, LEDC2012X120N, symbol LTST-C170KRKT:LTST-C170KRKT
- added R15: 50, symbol Device:R
- added R16, R18: 470, symbol Device:R
- C10: renamed from C7; value C -> 0.1u
- C9: renamed from C8; value C_Polarized -> 4.7u
Connections:
- net GND: now also C10.1, C9.1
- net +3.3V: now reaches R11.1, U4.6 (VDD), U4.7 (VREGIN)
- net +3.3V: now also C10.2, C9.2, LED5-GREEN.2 (A), LED6-RED.2 (A)
- net TX_RX: now reaches U3.11 (RXD)
- net RX_TX: now reaches U3.12 (TXD)
- net CD_SD: now reaches U3.18 (IO0)
- net EN: now reaches U3.2 (EN)
- net at U3.5 (IO6): now also R15.2
- net at U4.19 (~{RXT}/GPIO.3): now also R18.1
- net at U4.20 (~{TXT}/GPIO.2): now also R16.1
- new net: LED5-GREEN.1 (K), R16.2
- new net: LED6-RED.1 (K), R18.2
- new net SCLK: R15.1
- no-connect marks 0 -> 5
Other:
- note added: "USB MODULE"
- moved on the sheet: C10, C11, C9, R11, R12, R13, U3, U4, U5, U6
