File: Projects/Tutorial03-ESP32-IoT-4-layer-PCB/esp-32-c3-02.kicad_sch (KiCad schematic)
At the start: 30 parts, among them J3 GSD090012SEU, U3 ESP32-C3-WROOM-02-H4, U4 CP2102N-Axx-xQFN20, U5 USBLC6-2SC6, U6 W25Q32JVSSIQ

Commit message: 20260501
Changed lines of the file:
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@@
 	)
 	(junction
-		(at 141.478 134.62)
-		(diameter 0)
-		(color 0 0 0 0)
-	)
-	(junction
 		(at 59.69 35.56)
 		(diameter 0)
@@
 	)
 	(junction
-		(at 141.478 142.24)
-		(diameter 0)
-		(color 0 0 0 0)
-	)
-	(junction
 		(at 271.78 52.07)
 		(diameter 0)
@@
 	)
 	(junction
-		(at 141.478 137.16)
-		(diameter 0)
-		(color 0 0 0 0)
-	)
-	(junction
 		(at 242.57 45.72)
 		(diameter 0)
@@
 		(color 0 0 0 0)
 	)
-	(junction
-		(at 141.478 139.7)
-		(diameter 0)
-		(color 0 0 0 0)
-	)
 	(no_connect
 		(at 101.6 78.74)
@@
 	(wire
 		(pts
-			(xy 140.97 137.16) (xy 141.478 137.16)
-		)
-		(stroke
-			(width 0)
-			(type default)
-		)
-	)
-	(wire
-		(pts
 			(xy 22.86 76.2) (xy 35.56 76.2)
 		)
@@
 	(wire
 		(pts
-			(xy 141.478 139.7) (xy 144.78 139.7)
+			(xy 140.97 142.24) (xy 143.51 142.24)
 		)
 		(stroke
@@
 	(wire
 		(pts
-			(xy 141.478 142.24) (xy 144.78 142.24)
+			(xy 256.54 59.69) (xy 259.08 59.69)
 		)
 		(stroke
@@
 	(wire
 		(pts
-			(xy 256.54 59.69) (xy 259.08 59.69)
+			(xy 35.56 91.44) (xy 22.86 91.44)
 		)
 		(stroke
@@
 	(wire
 		(pts
-			(xy 35.56 91.44) (xy 22.86 91.44)
+			(xy 242.57 85.09) (xy 238.76 85.09)
 		)
 		(stroke
@@
 	(wire
 		(pts
-			(xy 242.57 85.09) (xy 238.76 85.09)
+			(xy 193.04 74.93) (xy 203.2 74.93)
 		)
 		(stroke
@@
 	(wire
 		(pts
-			(xy 193.04 74.93) (xy 203.2 74.93)
+			(xy 140.97 134.62) (xy 143.51 134.62)
 		)
 		(stroke
@@
 	(wire
 		(pts
-			(xy 140.97 134.62) (xy 141.478 134.62)
-		)
-		(stroke
-			(width 0)
-			(type default)
-		)
-	)
-	(wire
-		(pts
 			(xy 228.6 149.86) (xy 232.41 149.86)
 		)
@@
 	(wire
 		(pts
-			(xy 141.478 134.62) (xy 144.78 134.62)
-		)
-		(stroke
-			(width 0)
-			(type default)
-		)
-	)
-	(wire
-		(pts
 			(xy 22.86 91.44) (xy 22.86 95.25)
 		)
@@
 	(wire
 		(pts
-			(xy 140.97 139.7) (xy 141.478 139.7)
-		)
-		(stroke
-			(width 0)
-			(type default)
-		)
-	)
-	(wire
-		(pts
 			(xy 99.06 161.29) (xy 99.06 165.1)
 		)
@@
 	(wire
 		(pts
-			(xy 140.97 142.24) (xy 141.478 142.24)
-		)
-		(stroke
-			(width 0)
-			(type default)
-		)
-	)
-	(wire
-		(pts
 			(xy 99.06 165.1) (xy 99.06 168.91)
 		)
@@
 	(wire
 		(pts
+			(xy 140.97 139.7) (xy 143.51 139.7)
+		)
+		(stroke
+			(width 0)
+			(type default)
+		)
+	)
+	(wire
+		(pts
 			(xy 104.14 101.6) (xy 104.14 114.3)
 		)
@@
 	(wire
 		(pts
-			(xy 161.29 41.91) (xy 163.83 41.91)
+			(xy 140.97 137.16) (xy 143.51 137.16)
 		)
 		(stroke
@@
 	(wire
 		(pts
-			(xy 248.92 118.11) (xy 262.89 118.11)
+			(xy 161.29 41.91) (xy 163.83 41.91)
 		)
 		(stroke
@@
 	(wire
 		(pts
-			(xy 256.54 45.72) (xy 271.78 45.72)
+			(xy 248.92 118.11) (xy 262.89 118.11)
 		)
 		(stroke
@@
 	(wire
 		(pts
-			(xy 88.9 58.42) (xy 88.9 50.8)
+			(xy 256.54 45.72) (xy 271.78 45.72)
 		)
 		(stroke
@@
 	(wire
 		(pts
-			(xy 101.6 68.58) (xy 104.14 68.58)
+			(xy 88.9 58.42) (xy 88.9 50.8)
 		)
 		(stroke
@@
 	(wire
 		(pts
-			(xy 200.66 64.77) (xy 203.2 64.77)
+			(xy 101.6 68.58) (xy 104.14 68.58)
 		)
 		(stroke
@@
 	(wire
 		(pts
-			(xy 262.89 124.46) (xy 262.89 132.08)
+			(xy 200.66 64.77) (xy 203.2 64.77)
 		)
 		(stroke
@@
 	(wire
 		(pts
-			(xy 141.478 137.16) (xy 144.78 137.16)
+			(xy 262.89 124.46) (xy 262.89 132.08)
 		)
 		(stroke
@@
 	)
 	(label "SCL"
-		(at 144.78 139.7 0)
+		(at 143.51 139.7 0)
 		(effects
 			(font
@@
 	)
 	(label "SDA"
-		(at 144.78 142.24 0)
+		(at 143.51 142.24 0)
 		(effects
 			(font
@@
 	)
 	(label "MIC_OUT"
-		(at 144.78 134.62 0)
+		(at 143.51 134.62 0)
 		(effects
 			(font
@@
 	)
 	(label "PHOTO_C"
-		(at 144.78 137.16 0)
+		(at 143.51 137.16 0)
 		(effects
 			(font
@@
 	)
 	(sheet
-		(at 119.634 131.826)
+		(at 119.126 130.81)
 		(size 21.844 24.638)
 		(exclude_from_sim no)
@@
 		)
 		(property "Sheetname" "sensors"
-			(at 119.634 131.1144 0)
+			(at 119.126 130.0984 0)
 			(effects
 				(font
@@
 		)
 		(property "Sheetfile" "sensors.kicad_sch"
-			(at 119.634 157.0486 0)
+			(at 119.126 156.0326 0)
 			(effects
 				(font
@@
 		)
 		(pin "MIC_OUT" output
-			(at 141.478 134.62 0)
+			(at 140.97 134.62 0)
 			(effects
 				(font
@@
 		)
 		(pin "PHOTO_C" output
-			(at 141.478 137.16 0)
+			(at 140.97 137.16 0)
 			(effects
 				(font
@@
 		)
 		(pin "SCL" input
-			(at 141.478 139.7 0)
+			(at 140.97 139.7 0)
 			(effects
 				(font
@@
 		)
 		(pin "SDA" input
-			(at 141.478 142.24 0)
+			(at 140.97 142.24 0)
 			(effects
 				(font

Commit message: 20260516
Parts:
- U4: footprint Package_DFN_QFN:SiliconLabs_QFN-20-1EP_3x3mm_P0.5mm -> ESP32 Project Footprints:QFN20P400X400X100-21N
Changed lines of the file:
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@@
 			)
 		)
-		(property "Footprint" "Package_DFN_QFN:SiliconLabs_QFN-20-1EP_3x3mm_P0.5mm"
+		(property "Footprint" "ESP32 Project Footprints:QFN20P400X400X100-21N"
 			(at 120.65 113.03 0)
 			(effects

Commit message: 20260525
Parts:
- C12, C7, C9: footprint ESP32 Project Footprints:T491A -> Project-Footprints:T491A
- J3: footprint ESP32 Project Footprints:AMPHENOL_GSD090012SEU -> Project-Footprints:AMPHENOL_GSD090012SEU
- LED5-GREEN1: footprint ESP32 Project Footprints:LEDC2012X120N -> Project-Footprints:T491A
- LED6-RED1: footprint ESP32 Project Footprints:LEDC2012X120N -> Project-Footprints:LEDC2012X120N
- U3: footprint ESP32-C3-WROOM-02-H4:MODULE_ESP32-C3-WROOM-02-H4 -> Project-Footprints:MODULE_ESP32-C3-WROOM-02-H4
- U4: footprint ESP32 Project Footprints:QFN20P400X400X100-21N -> Project-Footprints:QFN20P400X400X100-21N
- U6: footprint W25Q32JVSSIQ:SOIC127P790X216-8N -> Package_SON:WSON-8-1EP_6x5mm_P1.27mm_EP3.4x4.3mm
Changed lines of the file:
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@@
 			)
 		)
-		(property "Footprint" "W25Q32JVSSIQ:SOIC127P790X216-8N"
+		(property "Footprint" "Package_SON:WSON-8-1EP_6x5mm_P1.27mm_EP3.4x4.3mm"
 			(at 78.74 157.48 0)
 			(effects
@@
 			)
 		)
-		(property "Footprint" "ESP32 Project Footprints:T491A"
+		(property "Footprint" "Project-Footprints:T491A"
 			(at 256.54 44.7548 0)
 			(effects
@@
 			)
 		)
-		(property "Footprint" "ESP32 Project Footprints:LEDC2012X120N"
+		(property "Footprint" "Project-Footprints:LEDC2012X120N"
 			(at 129.54 20.65 0)
 			(effects
@@
 			)
 		)
-		(property "Footprint" "ESP32 Project Footprints:T491A"
+		(property "Footprint" "Project-Footprints:T491A"
 			(at 241.3 117.1448 0)
 			(effects
@@
 			)
 		)
-		(property "Footprint" "ESP32 Project Footprints:T491A"
+		(property "Footprint" "Project-Footprints:T491A"
 			(at 72.39 34.5948 0)
 			(effects
@@
 			)
 		)
-		(property "Footprint" "ESP32 Project Footprints:LEDC2012X120N"
+		(property "Footprint" "Project-Footprints:T491A"
 			(at 129.54 5.41 0)
 			(effects
@@
 			)
 		)
-		(property "Footprint" "ESP32-C3-WROOM-02-H4:MODULE_ESP32-C3-WROOM-02-H4"
+		(property "Footprint" "Project-Footprints:MODULE_ESP32-C3-WROOM-02-H4"
 			(at 220.98 69.85 0)
 			(effects
@@
 			)
 		)
-		(property "Footprint" "ESP32 Project Footprints:QFN20P400X400X100-21N"
+		(property "Footprint" "Project-Footprints:QFN20P400X400X100-21N"
 			(at 120.65 113.03 0)
 			(effects
@@
 			)
 		)
-		(property "Footprint" "ESP32 Project Footprints:AMPHENOL_GSD090012SEU"
+		(property "Footprint" "Project-Footprints:AMPHENOL_GSD090012SEU"
 			(at 210.82 137.16 0)
 			(effects

Commit message: 20260525
Parts:
- added R17, R21: 4K7, Resistor_SMD:R_0805_2012Metric, symbol Device:R
Connections:
- net +3.3V: now also R17.1; no longer U6.3 (~{WP}(IO2)), U6.7 (~{HOLD}/~{RESET}(IO3))
- net GND: now also R21.2; no longer J3.8 (DAT1), J3.9 (DAT2)
- new net: R17.2, U6.3 (~{WP}(IO2)), U6.7 (~{HOLD}/~{RESET}(IO3))
- new net: J3.8 (DAT1), J3.9 (DAT2), R21.1
Changed lines of the file:
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@@
 	)
 	(junction
-		(at 262.89 132.08)
+		(at 59.69 35.56)
 		(diameter 0)
 		(color 0 0 0 0)
 	)
 	(junction
-		(at 59.69 35.56)
+		(at 99.06 165.1)
 		(diameter 0)
 		(color 0 0 0 0)
 	)
 	(junction
-		(at 99.06 165.1)
+		(at 232.41 147.32)
 		(diameter 0)
 		(color 0 0 0 0)
 	)
 	(junction
-		(at 29.21 157.48)
+		(at 237.49 118.11)
 		(diameter 0)
 		(color 0 0 0 0)
 	)
 	(junction
-		(at 232.41 147.32)
+		(at 99.06 149.86)
 		(diameter 0)
 		(color 0 0 0 0)
 	)
 	(junction
-		(at 229.87 132.08)
+		(at 262.89 132.08)
 		(diameter 0)
 		(color 0 0 0 0)
 	)
 	(junction
-		(at 237.49 118.11)
+		(at 242.57 52.07)
 		(diameter 0)
 		(color 0 0 0 0)
 	)
 	(junction
-		(at 99.06 149.86)
+		(at 29.21 157.48)
 		(diameter 0)
 		(color 0 0 0 0)
 	)
 	(junction
-		(at 242.57 52.07)
+		(at 229.87 132.08)
 		(diameter 0)
 		(color 0 0 0 0)
@@
 	(wire
 		(pts
+			(xy 257.81 132.08) (xy 262.89 132.08)
+		)
+		(stroke
+			(width 0)
+			(type default)
+		)
+	)
+	(wire
+		(pts
 			(xy 101.6 101.6) (xy 104.14 101.6)
 		)
@@
 	(wire
 		(pts
-			(xy 140.97 165.1) (xy 144.78 165.1)
+			(xy 29.21 152.4) (xy 29.21 157.48)
 		)
 		(stroke
@@
 	(wire
 		(pts
-			(xy 29.21 140.97) (xy 29.21 157.48)
+			(xy 140.97 165.1) (xy 144.78 165.1)
 		)
 		(stroke
@@
 	(wire
 		(pts
-			(xy 229.87 132.08) (xy 262.89 132.08)
-		)
-		(stroke
-			(width 0)
-			(type default)
-		)
-	)
-	(wire
-		(pts
 			(xy 58.42 152.4) (xy 60.96 152.4)
 		)
@@
 	(wire
 		(pts
+			(xy 229.87 132.08) (xy 250.19 132.08)
+		)
+		(stroke
+			(width 0)
+			(type default)
+		)
+	)
+	(wire
+		(pts
 			(xy 140.97 187.96) (xy 144.78 187.96)
 		)
@@
 	(wire
 		(pts
+			(xy 29.21 140.97) (xy 29.21 144.78)
+		)
+		(stroke
+			(width 0)
+			(type default)
+		)
+	)
+	(wire
+		(pts
 			(xy 161.29 41.91) (xy 163.83 41.91)
 		)
@@
 	(symbol
 		(lib_id "Device:R")
+		(at 29.21 148.59 0)
+		(unit 1)
+		(exclude_from_sim no)
+		(in_bom yes)
+		(on_board yes)
+		(dnp no)
+		(fields_autoplaced yes)
+		(property "Reference" "R17"
+			(at 31.75 147.3199 0)
+			(effects
+				(font
+					(size 1.27 1.27)
+				)
+				(justify left)
+			)
+		)
+		(property "Value" "4K7"
+			(at 31.75 149.8599 0)
+			(effects
+				(font
+					(size 1.27 1.27)
+				)
+				(justify left)
+			)
+		)
+		(property "Footprint" "Resistor_SMD:R_0805_2012Metric"
+			(at 27.432 148.59 90)
+			(effects
+				(font
+					(size 1.27 1.27)
+				)
+				(hide yes)
+			)
+		)
+		(property "Datasheet" "~"
+			(at 29.21 148.59 0)
+			(effects
+				(font
+					(size 1.27 1.27)
+				)
+				(hide yes)
+			)
+		)
+		(property "Description" "Resistor"
+			(at 29.21 148.59 0)
+			(effects
+				(font
+					(size 1.27 1.27)
+				)
+				(hide yes)
+			)
+		)
+		(pin "2"
+		)
+		(pin "1"
+		)
+		(instances
+			(project "Tutorial03-ESP32-IoT-4-layer-PCB"
+				(path "/49253bfd-5dbd-467b-ba3c-7c0c524516c8/088a6c03-a50a-4238-8650-576912e1e4b8"
+					(reference "R17")
+					(unit 1)
+				)
+			)
+		)
+	)
+	(symbol
+		(lib_id "Device:R")
 		(at 22.86 83.82 0)
 		(unit 1)
@@
 					(unit 1)
 				)
+			)
+		)
+	)
+	(symbol
+		(lib_id "Device:R")
+		(at 254 132.08 90)
+		(unit 1)
+		(exclude_from_sim no)
+		(in_bom yes)
+		(on_board yes)
+		(dnp no)
+		(property "Reference" "R21"
+			(at 251.714 129.54 90)
+			(effects
+				(font
+					(size 1.27 1.27)
+				)
+			)
+		)
+		(property "Value" "4K7"
+			(at 257.302 129.54 90)
+			(effects
+				(font
+					(size 1.27 1.27)
+				)
+			)
+		)
+		(property "Footprint" "Resistor_SMD:R_0805_2012Metric"
+			(at 254 133.858 90)
+			(effects
+				(font
+					(size 1.27 1.27)
+				)
+				(hide yes)
+			)
+		)
+		(property "Datasheet" "~"
+			(at 254 132.08 0)
+			(effects
+				(font
+					(size 1.27 1.27)
+				)
+				(hide yes)
+			)
+		)
+		(property "Description" "Resistor"
+			(at 254 132.08 0)
+			(effects
+				(font
+					(size 1.27 1.27)
+				)
+				(hide yes)
+			)
+		)
+		(pin "2"
+		)
+		(pin "1"
+		)
+		(instances
+			(project "Tutorial03-ESP32-IoT-4-layer-PCB"
+				(path "/49253bfd-5dbd-467b-ba3c-7c0c524516c8/088a6c03-a50a-4238-8650-576912e1e4b8"
+					(reference "R21")
+					(unit 1)
+				)

Commit message: 20260602
Parts:
- TP1: footprint Connector_PinHeader_2.54mm:PinHeader_1x04_P2.54mm_Vertical -> TestPoint:TestPoint_Pad_D1.0mm
Changed lines of the file:
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@@
 			)
 		)
-		(property "Footprint" "Connector_PinHeader_2.54mm:PinHeader_1x04_P2.54mm_Vertical"
+		(property "Footprint" "TestPoint:TestPoint_Pad_D1.0mm"
 			(at 161.29 26.67 0)
 			(effects

Commit message: 20260620
Parts:
- LED5G1: renamed from LED5-GREEN1; footprint Project-Footprints:T491A -> Project-Footprints:LEDC2012X120N
- renumbered LED6-RED1 to LED6R1
Changed lines of the file:
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@@
 		(on_board yes)
 		(dnp no)
-		(property "Reference" "LED6-RED1"
+		(property "Reference" "LED6R1"
 			(at 120.142 109.22 0)
 			(effects
@@
 			(project "Tutorial03-ESP32-IoT-4-layer-PCB"
 				(path "/49253bfd-5dbd-467b-ba3c-7c0c524516c8/088a6c03-a50a-4238-8650-576912e1e4b8"
-					(reference "LED6-RED1")
+					(reference "LED6R1")
 					(unit 1)
 				)
@@
 		(on_board yes)
 		(dnp no)
-		(property "Reference" "LED5-GREEN1"
+		(property "Reference" "LED5G1"
 			(at 121.92 94.234 0)
 			(effects
@@
 			)
 		)
-		(property "Footprint" "Project-Footprints:T491A"
+		(property "Footprint" "Project-Footprints:LEDC2012X120N"
 			(at 129.54 5.41 0)
 			(effects
@@
 			(project "Tutorial03-ESP32-IoT-4-layer-PCB"
 				(path "/49253bfd-5dbd-467b-ba3c-7c0c524516c8/088a6c03-a50a-4238-8650-576912e1e4b8"
-					(reference "LED5-GREEN1")
-					(unit 1)
-				)
+					(reference "LED5G1")
+					(unit 1)
+				)
