File: Projects/Tutorial03-ESP32-IoT-4-layer-PCB/esp-32-c3-02.kicad_sch (KiCad schematic)
At the start: 32 parts, among them J3 GSD090012SEU, U3 ESP32-C3-WROOM-02-H4, U4 CP2102N-Axx-xQFN20, U5 USBLC6-2SC6, U6 W25Q32JVSSIQ

Commit message: 20260920
Parts:
- U4: footprint Project-Footprints:QFN20P400X400X100-21N -> Project-Footprints:QFN-20_L3.0-W3.0-P0.50-BL-EP1.7_EFM8BB21F16G
Changed lines of the file:
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@@
 			)
 		)
-		(property "Footprint" "Project-Footprints:QFN20P400X400X100-21N"
+		(property "Footprint" "Project-Footprints:QFN-20_L3.0-W3.0-P0.50-BL-EP1.7_EFM8BB21F16G"
 			(at 120.65 113.03 0)
 			(hide yes)
