File: Projects/Tutorial03-ESP32-IoT-4-layer-PCB/sensors.kicad_sch (KiCad schematic)
At the start: 0 parts

Commit message: 20260315
Parts:
- added C15, C16, C18, C20: 0.1u, symbol Device:C
- added MK1: CMC-5042PF-AC, CMC-5042PF-AC:CUI_CMC-5042PF-AC, symbol CMC-5042PF-AC:CMC-5042PF-AC
- added Q1: TEMT6000X01, TEMT6000X01:TRANS_TEMT6000X01, symbol TEMT6000X01:TEMT6000X01
- added R23, R27, R29, R30: 10K, symbol Device:R
- added R24, R25: 4K7, symbol Device:R
- added R26, R28: 2K, symbol Device:R
- added R31: 100K, symbol Device:R
- added U2: MAX4466EXK, MAX4466EXK:SOT65P210X110-5N, symbol MAX4466EXK:MAX4466EXK
- added U7: BME280, BME280:PSON65P250X250X100-8N, symbol BME280:BME280
Connections:
- new net: C16.2, R26.2, R28.1
- new net: MK1.OUT, R27.2, R28.2, R29.1, U2.1 (IN+)
- new net +3.3V: C15.1, C18.1, R23.1, R24.1, R25.1, R26.1, R27.1, U2.5 (VCC), U7.2 (CSB), U7.6 (VDDIO), U7.8 (VDD)
- new net GND: C15.2, C16.1, C18.2, C20.1, MK1.GND, Q1.1, R29.2, R30.1, R30.2, R31.1, U2.2 (GND), U2.3 (IN-), U7.1 (GND), U7.5 (SDO), U7.7 (GND)
- new net MIC_OUT: C20.2, R31.2, U2.4 (OUT)
- new net PHOTO_C: Q1.3, R23.2
- new net SCL: R25.2, U7.4 (SCK)
- new net SDA: R24.2, U7.3 (SDI)
Other:
- note added: "MICROPHONE AND PREAMPLIFIER"
- note added: "PHOTO SENSOR"
- note added: "TEMPERATURE AND PRESSURE SENSOR"

Commit message: 20260425
Parts:
- C15, C16, C18, C20: footprint (none) -> Capacitor_SMD:C_0805_2012Metric
- MK1: footprint CMC-5042PF-AC:CUI_CMC-5042PF-AC -> ESP32 Project Footprints:CUI_CMC-5042PF-AC
- Q1: footprint TEMT6000X01:TRANS_TEMT6000X01 -> ESP32 Project Footprints:TRANS_TEMT6000X01
- R23, R24, R25, R26, R27, R28, R29, R30, R31: footprint (none) -> Resistor_SMD:R_0805_2012Metric
Changed lines of the file:
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@@
 			)
 		)
-		(property "Footprint" ""
+		(property "Footprint" "Resistor_SMD:R_0805_2012Metric"
 			(at 196.342 49.53 90)
 			(effects
@@
 			)
 		)
-		(property "Footprint" ""
+		(property "Footprint" "Resistor_SMD:R_0805_2012Metric"
 			(at 174.498 102.87 90)
 			(effects
@@
 			)
 		)
-		(property "Footprint" ""
+		(property "Footprint" "Resistor_SMD:R_0805_2012Metric"
 			(at 229.87 142.748 90)
 			(effects
@@
 			)
 		)
-		(property "Footprint" ""
+		(property "Footprint" "Capacitor_SMD:C_0805_2012Metric"
 			(at 263.8552 130.81 0)
 			(effects
@@
 			)
 		)
-		(property "Footprint" ""
+		(property "Footprint" "Capacitor_SMD:C_0805_2012Metric"
 			(at 163.83 110.1852 0)
 			(effects
@@
 			)
 		)
-		(property "Footprint" ""
+		(property "Footprint" "Resistor_SMD:R_0805_2012Metric"
 			(at 201.168 130.81 90)
 			(effects
@@
 			)
 		)
-		(property "Footprint" ""
+		(property "Footprint" "Resistor_SMD:R_0805_2012Metric"
 			(at 42.672 50.8 90)
 			(effects
@@
 			)
 		)
-		(property "Footprint" ""
+		(property "Footprint" "Resistor_SMD:R_0805_2012Metric"
 			(at 174.498 114.3 90)
 			(effects
@@
 			)
 		)
-		(property "Footprint" "CMC-5042PF-AC:CUI_CMC-5042PF-AC"
+		(property "Footprint" "ESP32 Project Footprints:CUI_CMC-5042PF-AC"
 			(at 139.7 124.46 0)
 			(effects
@@
 			)
 		)
-		(property "Footprint" ""
+		(property "Footprint" "Resistor_SMD:R_0805_2012Metric"
 			(at 51.562 50.8 90)
 			(effects
@@
 			)
 		)
-		(property "Footprint" ""
+		(property "Footprint" "Resistor_SMD:R_0805_2012Metric"
 			(at 188.468 128.27 90)
 			(effects
@@
 			)
 		)
-		(property "Footprint" ""
+		(property "Footprint" "Resistor_SMD:R_0805_2012Metric"
 			(at 188.468 114.3 90)
 			(effects
@@
 			)
 		)
-		(property "Footprint" "TEMT6000X01:TRANS_TEMT6000X01"
+		(property "Footprint" "ESP32 Project Footprints:TRANS_TEMT6000X01"
 			(at 185.42 58.42 0)
 			(effects
@@
 			)
 		)
-		(property "Footprint" ""
+		(property "Footprint" "Capacitor_SMD:C_0805_2012Metric"
 			(at 105.1052 64.77 0)
 			(effects
@@
 			)
 		)
-		(property "Footprint" ""
+		(property "Footprint" "Capacitor_SMD:C_0805_2012Metric"
 			(at 233.68 148.2852 0)
 			(effects

Commit message: 20260501
Changed lines of the file:
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@@
-	(text_box ""
-		(exclude_from_sim no)
-		(at 129.54 87.376 0)
-		(size 145.034 70.866)
-		(margins 0.9525 0.9525 0.9525 0.9525)
-		(stroke
-			(width 0)
-			(type solid)
-		)
-		(fill
-			(type none)
-		)
-		(effects
-			(font
-				(size 1.27 1.27)
-			)
-			(justify left top)
-		)
-	)
 	(text_box ""
 		(exclude_from_sim no)
@@
 	)
 	(junction
-		(at 262.89 116.84)
-		(diameter 0)
-		(color 0 0 0 0)
-	)
-	(junction
 		(at 152.4 127)
 		(diameter 0)
@@
 	)
 	(junction
-		(at 262.89 104.14)
-		(diameter 0)
-		(color 0 0 0 0)
-	)
-	(junction
 		(at 104.14 71.12)
 		(diameter 0)
@@
 	)
 	(junction
+		(at 262.89 116.84)
+		(diameter 0)
+		(color 0 0 0 0)
+	)
+	(junction
 		(at 186.69 140.97)
 		(diameter 0)
@@
 	(wire
 		(pts
-			(xy 262.89 116.84) (xy 262.89 104.14)
-		)
-		(stroke
-			(width 0)
-			(type default)
-		)
-	)
-	(wire
-		(pts
 			(xy 172.72 106.68) (xy 172.72 109.22)
 		)
@@
 	(wire
 		(pts
-			(xy 262.89 104.14) (xy 262.89 102.87)
-		)
-		(stroke
-			(width 0)
-			(type default)
-		)
-	)
-	(wire
-		(pts
 			(xy 199.39 140.97) (xy 208.28 140.97)
 		)
@@
 	(wire
 		(pts
-			(xy 64.77 74.93) (xy 64.77 66.04)
-		)
-		(stroke
-			(width 0)
-			(type default)
-		)
-	)
-	(wire
-		(pts
 			(xy 53.34 46.99) (xy 53.34 44.45)
 		)
@@
 	(wire
 		(pts
-			(xy 64.77 66.04) (xy 68.58 66.04)
+			(xy 64.77 66.04) (xy 64.77 68.58)
 		)
 		(stroke
@@
 	(wire
 		(pts
+			(xy 68.58 66.04) (xy 64.77 66.04)
+		)
+		(stroke
+			(width 0)
+			(type default)
+		)
+	)
+	(wire
+		(pts
 			(xy 199.39 134.62) (xy 199.39 140.97)
 		)
@@
 		(pts
 			(xy 220.98 140.97) (xy 226.06 140.97)
+		)
+		(stroke
+			(width 0)
+			(type default)
+		)
+	)
+	(wire
+		(pts
+			(xy 262.89 101.6) (xy 262.89 116.84)
 		)
 		(stroke
@@
 	(symbol
 		(lib_id "power:+3.3V")
-		(at 262.89 104.14 0)
+		(at 262.89 101.6 0)
 		(unit 1)
 		(exclude_from_sim no)
@@
 		(fields_autoplaced yes)
 		(property "Reference" "#PWR040"
-			(at 262.89 107.95 0)
+			(at 262.89 105.41 0)
 			(effects
 				(font
@@
 		)
 		(property "Value" "+3.3V"
-			(at 262.89 99.06 0)
+			(at 262.89 96.52 0)
 			(effects
 				(font
@@
 		)
 		(property "Footprint" ""
-			(at 262.89 104.14 0)
+			(at 262.89 101.6 0)
 			(effects
 				(font
@@
 		)
 		(property "Datasheet" ""
-			(at 262.89 104.14 0)
+			(at 262.89 101.6 0)
 			(effects
 				(font
@@
 		)
 		(property "Description" "Power symbol creates a global label with name \"+3.3V\""
-			(at 262.89 104.14 0)
+			(at 262.89 101.6 0)
 			(effects
 				(font
@@
 	(symbol
 		(lib_id "power:GND")
-		(at 64.77 74.93 0)
+		(at 64.77 68.58 0)
 		(unit 1)
 		(exclude_from_sim no)
@@
 		(fields_autoplaced yes)
 		(property "Reference" "#PWR035"
-			(at 64.77 81.28 0)
+			(at 64.77 74.93 0)
 			(effects
 				(font
@@
 		)
 		(property "Value" "GND"
-			(at 64.77 80.01 0)
+			(at 64.77 73.66 0)
 			(effects
 				(font
@@
 		)
 		(property "Footprint" ""
-			(at 64.77 74.93 0)
+			(at 64.77 68.58 0)
 			(effects
 				(font
@@
 		)
 		(property "Datasheet" ""
-			(at 64.77 74.93 0)
+			(at 64.77 68.58 0)
 			(effects
 				(font
@@
 		)
 		(property "Description" "Power symbol creates a global label with name \"GND\" , ground"
-			(at 64.77 74.93 0)
-			(effects
-				(font
+			(at 64.77 68.58 0)
+			(effects
+				(font

Commit message: 20260525
Parts:
- MK1: footprint ESP32 Project Footprints:CUI_CMC-5042PF-AC -> Project-Footprints:CUI_CMC-5042PF-AC
- Q1: footprint ESP32 Project Footprints:TRANS_TEMT6000X01 -> Project-Footprints:TRANS_TEMT6000X01
- U2: footprint MAX4466EXK:SOT65P210X110-5N -> Project-Footprints:SOT65P210X110-5N
- U7: footprint BME280:PSON65P250X250X100-8N -> Project-Footprints:PSON65P250X250X100-8N
Changed lines of the file:
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@@
 			)
 		)
-		(property "Footprint" "ESP32 Project Footprints:CUI_CMC-5042PF-AC"
+		(property "Footprint" "Project-Footprints:CUI_CMC-5042PF-AC"
 			(at 139.7 124.46 0)
 			(effects
@@
 			)
 		)
-		(property "Footprint" "BME280:PSON65P250X250X100-8N"
+		(property "Footprint" "Project-Footprints:PSON65P250X250X100-8N"
 			(at 83.82 60.96 0)
 			(effects
@@
 			)
 		)
-		(property "Footprint" "MAX4466EXK:SOT65P210X110-5N"
+		(property "Footprint" "Project-Footprints:SOT65P210X110-5N"
 			(at 228.6 124.46 0)
 			(effects
@@
 			)
 		)
-		(property "Footprint" "ESP32 Project Footprints:TRANS_TEMT6000X01"
+		(property "Footprint" "Project-Footprints:TRANS_TEMT6000X01"
 			(at 185.42 58.42 0)
 			(effects

Commit message: 20260525
Parts:
- added R35: 4K7, Resistor_SMD:R_0805_2012Metric, symbol Device:R
Connections:
- net GND: now also R35.2; no longer U7.5 (SDO)
- new net: R35.1, U7.5 (SDO)
Changed lines of the file:
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@@
+	(wire
+		(pts
+			(xy 53.34 66.04) (xy 68.58 66.04)
+		)
+		(stroke
+			(width 0)
+			(type default)
+		)
+	)
 	(wire
 		(pts
@@
 	(wire
 		(pts
+			(xy 53.34 74.93) (xy 53.34 77.47)
+		)
+		(stroke
+			(width 0)
+			(type default)
+		)
+	)
+	(wire
+		(pts
 			(xy 262.89 132.08) (xy 262.89 144.78)
 		)
@@
 	(wire
 		(pts
+			(xy 53.34 66.04) (xy 53.34 67.31)
+		)
+		(stroke
+			(width 0)
+			(type default)
+		)
+	)
+	(wire
+		(pts
 			(xy 172.72 109.22) (xy 172.72 110.49)
 		)
@@
 	(wire
 		(pts
-			(xy 64.77 66.04) (xy 64.77 68.58)
-		)
-		(stroke
-			(width 0)
-			(type default)
-		)
-	)
-	(wire
-		(pts
 			(xy 64.77 40.64) (xy 64.77 44.45)
 		)
@@
 		(pts
 			(xy 233.68 140.97) (xy 238.76 140.97)
-		)
-		(stroke
-			(width 0)
-			(type default)
-		)
-	)
-	(wire
-		(pts
-			(xy 68.58 66.04) (xy 64.77 66.04)
 		)
 		(stroke
@@
 	(symbol
 		(lib_id "Device:R")
+		(at 53.34 71.12 0)
+		(unit 1)
+		(exclude_from_sim no)
+		(in_bom yes)
+		(on_board yes)
+		(dnp no)
+		(fields_autoplaced yes)
+		(property "Reference" "R35"
+			(at 55.88 69.8499 0)
+			(effects
+				(font
+					(size 1.27 1.27)
+				)
+				(justify left)
+			)
+		)
+		(property "Value" "4K7"
+			(at 55.88 72.3899 0)
+			(effects
+				(font
+					(size 1.27 1.27)
+				)
+				(justify left)
+			)
+		)
+		(property "Footprint" "Resistor_SMD:R_0805_2012Metric"
+			(at 51.562 71.12 90)
+			(effects
+				(font
+					(size 1.27 1.27)
+				)
+				(hide yes)
+			)
+		)
+		(property "Datasheet" "~"
+			(at 53.34 71.12 0)
+			(effects
+				(font
+					(size 1.27 1.27)
+				)
+				(hide yes)
+			)
+		)
+		(property "Description" "Resistor"
+			(at 53.34 71.12 0)
+			(effects
+				(font
+					(size 1.27 1.27)
+				)
+				(hide yes)
+			)
+		)
+		(pin "2"
+		)
+		(pin "1"
+		)
+		(instances
+			(project "Tutorial03-ESP32-IoT-4-layer-PCB"
+				(path "/49253bfd-5dbd-467b-ba3c-7c0c524516c8/088a6c03-a50a-4238-8650-576912e1e4b8/82f04113-e066-48bd-98ff-7ce17d570a0d"
+					(reference "R35")
+					(unit 1)
+				)
+			)
+		)
+	)
+	(symbol
+		(lib_id "Device:R")
 		(at 172.72 114.3 0)
 		(mirror y)
@@
 	(symbol
 		(lib_id "power:GND")
-		(at 64.77 68.58 0)
+		(at 53.34 77.47 0)
 		(unit 1)
 		(exclude_from_sim no)
@@
 		(fields_autoplaced yes)
 		(property "Reference" "#PWR035"
-			(at 64.77 74.93 0)
+			(at 53.34 83.82 0)
 			(effects
 				(font
@@
 		)
 		(property "Value" "GND"
-			(at 64.77 73.66 0)
+			(at 53.34 82.55 0)
 			(effects
 				(font
@@
 		)
 		(property "Footprint" ""
-			(at 64.77 68.58 0)
+			(at 53.34 77.47 0)
 			(effects
 				(font
@@
 		)
 		(property "Datasheet" ""
-			(at 64.77 68.58 0)
+			(at 53.34 77.47 0)
 			(effects
 				(font
@@
 		)
 		(property "Description" "Power symbol creates a global label with name \"GND\" , ground"
-			(at 64.77 68.58 0)
-			(effects
-				(font
+			(at 53.34 77.47 0)
+			(effects
+				(font
