File: Projects/Tutorial03-ESP32-IoT-4-layer-PCB/sensors.kicad_sch (KiCad schematic)
At the start: 20 parts, among them Q1 TEMT6000X01, U2 MAX4466EXK, U7 BME280

Commit message: 20260704
Parts:
- U7: DESCRIPTION Integrated pressure, humidity and temperature sensor; 8-pin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 -> (none)

Commit message: 20260905
Changed lines of the file:
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@@
+		)
+	)
+	(text_box ""
+		(exclude_from_sim no)
+		(at 125.73 83.82 0)
+		(size 152.4 75.565)
+		(margins 0.9525 0.9525 0.9525 0.9525)
+		(stroke
+			(width 0)
+			(type solid)
+		)
+		(fill
+			(type none)
+		)
+		(effects
+			(font
+				(size 1.27 1.27)
+			)
+			(justify left top)
 		)
 	)
