File: Projects/Tutorial03-ESP32-IoT-4-layer-PCB/Tutorial03-ESP32-IoT-4-layer-PCB.kicad_pcb (KiCad board)
At the start: 4 copper layers, 0 parts

Commit message: 20260525
Parts:
- added C1: 0.1u, Capacitor_SMD:C_0805_2012Metric, F.Cu at (88.6, 41.2)
- added C10: 0.1u, Capacitor_SMD:C_0805_2012Metric, F.Cu at (54.5, 26.8)
- added C11: 1u, Capacitor_SMD:C_0805_2012Metric, F.Cu at (54.5, 29.8)
- added C12: 10u, Project-Footprints:T491A, F.Cu at (46.9, 62.7)
- added C13: 0.1u, Capacitor_SMD:C_0805_2012Metric, F.Cu at (54.5, 32.9)
- added C14: 0.1u, Capacitor_SMD:C_0805_2012Metric, F.Cu at (54.5, 35.9)
- added C15: 0.1u, Capacitor_SMD:C_0805_2012Metric, F.Cu at (76.7, 55.2)
- added C16: 0.1u, Capacitor_SMD:C_0805_2012Metric, F.Cu at (76.7, 58.2)
- added C17: 0.1u, Capacitor_SMD:C_0805_2012Metric, F.Cu at (28.7, 88.3)
- added C18: 0.1u, Capacitor_SMD:C_0805_2012Metric, F.Cu at (76.7, 61.2)
- added C19: 0.1u, Capacitor_SMD:C_0805_2012Metric, F.Cu at (28.7, 91.3)
- added C2: 0.1u, Capacitor_SMD:C_0805_2012Metric, F.Cu at (88.6, 44.2)
- added C20: 0.1u, Capacitor_SMD:C_0805_2012Metric, F.Cu at (76.7, 64.2)
- added C3: 10u, Project-Footprints:T491A, F.Cu at (82.9, 42.0)
- added C4: 10u, Project-Footprints:T491A, F.Cu at (82.9, 46.6)
- added C5: 0.1u, Capacitor_SMD:C_0805_2012Metric, F.Cu at (88.6, 47.2)
- added C6: 1u, Capacitor_SMD:C_0805_2012Metric, F.Cu at (88.6, 50.2)
- added C7: 10u, Project-Footprints:T491A, F.Cu at (46.9, 53.4)
- added C8: 0.1u, Capacitor_SMD:C_0805_2012Metric, F.Cu at (54.5, 23.8)
- added C9: 4.7u, Project-Footprints:T491A, F.Cu at (46.9, 58.0)
- added F1: 0ZCH0110AF2E, Project-Footprints:FUSC3226X100N, F.Cu at (92.1, 24.5)
- added J1: SS-52400-002, Project-Footprints:BELFUSE_SS-52400-002, F.Cu at (71.3, 31.4)
- added J2: B2B-PH-SM4-TB, Project-Footprints:JST_B2B-PH-SM4-TB, F.Cu at (84.3, 25.6)
- added J3: GSD090012SEU, Project-Footprints:AMPHENOL_GSD090012SEU, F.Cu at (37.1, 37.8)
- added J4: Conn_01x04_Pin, Connector_PinHeader_2.54mm:PinHeader_1x04_P2.54mm_Vertical, F.Cu at (28.8, 76.9)
- added J5: Conn_01x05_Pin, Connector_PinHeader_2.54mm:PinHeader_1x05_P2.54mm_Vertical, F.Cu at (24.2, 76.9)
- added LED1-RED1: LTST-C170KRKT, Project-Footprints:LEDC2012X120N, F.Cu at (76.9, 38.3)
- added LED2-GREEN1: LTST-C170GKT, Project-Footprints:LEDC2012X120N, F.Cu at (76.9, 41.6)
- added LED2-RED1: LTST-C170KRKT, Project-Footprints:LEDC2012X120N, F.Cu at (76.9, 45.0)
- added LED3-BLUE1: LTST-C170TBKT, Project-Footprints:LEDC2012X120N, F.Cu at (76.9, 48.3)
- added LED5-GREEN1: LTST-C170GKT, Project-Footprints:T491A, F.Cu at (46.9, 67.3)
- added LED6-RED1: LTST-C170KRKT, Project-Footprints:LEDC2012X120N, F.Cu at (52.8, 69.1)
- added MK1: CMC-5042PF-AC, Project-Footprints:CUI_CMC-5042PF-AC, F.Cu at (78.3, 69.5)
- added Q1: TEMT6000X01, Project-Footprints:TRANS_TEMT6000X01, F.Cu at (69.4, 70.3)
- added Q2: BC817, Package_TO_SOT_SMD:SOT-23, F.Cu at (33.6, 76.8)
- added Q3: BC817, Package_TO_SOT_SMD:SOT-23, F.Cu at (33.6, 81.3)
- added R1: 10K, Resistor_SMD:R_0805_2012Metric, F.Cu at (67.9, 38.1)
- added R10: 470, Resistor_SMD:R_0805_2012Metric, F.Cu at (72.3, 49.9)
- added R11: 1k, Resistor_SMD:R_0805_2012Metric, F.Cu at (52.7, 52.5)
- added R12: 22K1, Resistor_SMD:R_0805_2012Metric, F.Cu at (52.7, 55.5)
- added R13: 47K5, Resistor_SMD:R_0805_2012Metric, F.Cu at (52.7, 58.4)
- added R14: 50, Resistor_SMD:R_0805_2012Metric, F.Cu at (52.7, 61.4)
- added R15: 50, Resistor_SMD:R_0805_2012Metric, F.Cu at (57.1, 52.5)
- added R16: 470, Resistor_SMD:R_0805_2012Metric, F.Cu at (57.1, 55.5)
- added R17: 4K7, Resistor_SMD:R_0805_2012Metric, F.Cu at (57.1, 58.4)
- added R18: 470, Resistor_SMD:R_0805_2012Metric, F.Cu at (57.1, 61.4)
- added R19: 10K, Resistor_SMD:R_0805_2012Metric, F.Cu at (61.5, 52.5)
- added R2: 10K, Resistor_SMD:R_0805_2012Metric, F.Cu at (67.9, 41.0)
- added R20: 50, Resistor_SMD:R_0805_2012Metric, F.Cu at (61.5, 55.5)
- added R21: 4K7, Resistor_SMD:R_0805_2012Metric, F.Cu at (61.5, 58.4)
- added R22: 50, Resistor_SMD:R_0805_2012Metric, F.Cu at (61.5, 61.4)
- added R23: 10K, Resistor_SMD:R_0805_2012Metric, F.Cu at (67.9, 55.2)
- added R24: 4K7, Resistor_SMD:R_0805_2012Metric, F.Cu at (67.9, 58.1)
- added R25: 4K7, Resistor_SMD:R_0805_2012Metric, F.Cu at (67.9, 61.1)
- added R26: 2K, Resistor_SMD:R_0805_2012Metric, F.Cu at (67.9, 64.0)
- added R27: 10K, Resistor_SMD:R_0805_2012Metric, F.Cu at (67.9, 67.0)
- added R28: 2K, Resistor_SMD:R_0805_2012Metric, F.Cu at (72.3, 55.2)
- added R29: 10K, Resistor_SMD:R_0805_2012Metric, F.Cu at (72.3, 58.1)
- added R3: 5K1, Resistor_SMD:R_0805_2012Metric, F.Cu at (67.9, 44.0)
- added R30: 10K, Resistor_SMD:R_0805_2012Metric, F.Cu at (72.3, 61.1)
- added R31: 100K, Resistor_SMD:R_0805_2012Metric, F.Cu at (72.3, 64.0)
- added R32: 10K, Resistor_SMD:R_0805_2012Metric, F.Cu at (38.2, 76.1)
- added R33: 10K, Resistor_SMD:R_0805_2012Metric, F.Cu at (38.2, 79.0)
- added R34: 10K, Resistor_SMD:R_0805_2012Metric, F.Cu at (38.2, 82.0)
- added R35: 4K7, Resistor_SMD:R_0805_2012Metric, F.Cu at (72.3, 67.0)
- added R4: 5K1, Resistor_SMD:R_0805_2012Metric, F.Cu at (67.9, 46.9)
- added R5: 2K, Resistor_SMD:R_0805_2012Metric, F.Cu at (67.9, 49.9)
- added R6: 20K, Resistor_SMD:R_0805_2012Metric, F.Cu at (72.3, 38.1)
- added R7: 470, Resistor_SMD:R_0805_2012Metric, F.Cu at (72.3, 41.0)
- added R8: 470, Resistor_SMD:R_0805_2012Metric, F.Cu at (72.3, 44.0)
- added R9: 470, Resistor_SMD:R_0805_2012Metric, F.Cu at (72.3, 46.9)
- added S1: USLPT2819DT2TR, Project-Footprints:SW_USLPT2819DT2TR, F.Cu at (34.0, 85.2)
- added S2: USLPT2819DT2TR, Project-Footprints:SW_USLPT2819DT2TR, F.Cu at (34.0, 88.7)
- added TP1: Test MISO_DI, Connector_PinHeader_2.54mm:PinHeader_1x04_P2.54mm_Vertical, F.Cu at (59.0, 24.6)
- added TP2: Test MISO_DO, TestPoint:TestPoint_Pad_D1.0mm, F.Cu at (53.8, 38.9)
- added TP3: Test SCKL, TestPoint:TestPoint_Pad_D1.0mm, F.Cu at (53.8, 41.9)
- added TP4: Test CS_SD, TestPoint:TestPoint_Pad_D1.0mm, F.Cu at (53.8, 45.0)
- added TP5: Test CS, TestPoint:TestPoint_Pad_D1.0mm, F.Cu at (53.8, 48.0)
- added U1: MCP73871, Package_DFN_QFN:QFN-20-1EP_4x4mm_P0.5mm_EP2.5x2.5mm, F.Cu at (91.8, 35.1)
- added U2: MAX4466EXK, Project-Footprints:SOT65P210X110-5N, F.Cu at (81.7, 55.6)
- added U3: ESP32-C3-WROOM-02-H4, Project-Footprints:MODULE_ESP32-C3-WROOM-02-H4, F.Cu at (33.1, 61.8)
- added U4: CP2102N-Axx-xQFN20, Project-Footprints:QFN20P400X400X100-21N, F.Cu at (58.9, 47.0)
- added U5: USBLC6-2SC6, Package_TO_SOT_SMD:SOT-23-6, F.Cu at (53.0, 65.2)
- added U6: W25Q32JVSSIQ, Package_SON:WSON-8-1EP_6x5mm_P1.27mm_EP3.4x4.3mm, F.Cu at (59.6, 40.6)
- added U7: BME280, Project-Footprints:PSON65P250X250X100-8N, F.Cu at (81.0, 59.5)
- added VR1: LM1117MPX-3.3, Project-Footprints:VREG_LM1117MPX-3.3, F.Cu at (83.8, 35.8)

Commit message: 20260525
Parts:
- moved R11 93.4 mm to (141.2, 82.5)
- moved R12 93.4 mm to (141.2, 85.5)
- moved R13 93.4 mm to (141.2, 88.4)
- moved R15 93.4 mm to (145.6, 82.5)
- moved R16 93.4 mm to (145.6, 85.5)
- moved R17 93.4 mm to (145.6, 88.4)
- moved R19 93.4 mm to (150.0, 82.5)
- moved R20 93.4 mm to (150.0, 85.5)
- moved R21 93.4 mm to (150.0, 88.4)
- moved R14 93.4 mm to (141.2, 91.3)
- moved R18 93.4 mm to (145.6, 91.3)
- moved R22 93.4 mm to (150.0, 91.3)
- moved U2 81.4 mm to (162.8, 62.6)
- moved U7 81.4 mm to (162.1, 66.6)
- moved U1 72.7 mm to (163.7, 24.8)
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
Commit message: 20260530
Parts:
- moved J3 198.9 mm to (216.9, 122.7)
- moved U3 184.5 mm to (216.0, 86.1)
- moved C13 178.0 mm to (217.6, 104.2), turned to 180 degrees
- moved C12 164.5 mm to (206.1, 104.2)
- moved C7 159.3 mm to (201.4, 92.2)
- moved C8 157.2 mm to (202.3, 77.2)
- moved C18 144.6 mm to (136.8, -82.9)
- moved C19 144.6 mm to (15.4, -46.1)
- moved C6 144.6 mm to (148.7, -93.9)
- moved J1 144.6 mm to (59.4, -112.7)
- moved J4 144.6 mm to (16.9, -67.2)
- moved J5 144.6 mm to (12.3, -67.2)
- moved LED2-RED1 144.6 mm to (136.9, -99.1)
- moved Q1 144.6 mm to (129.4, -73.8)
- moved Q2 144.6 mm to (35.0, -64.4)
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
Commit message: 20260602
Parts:
- TP1: footprint Connector_PinHeader_2.54mm:PinHeader_1x04_P2.54mm_Vertical -> TestPoint:TestPoint_Pad_D1.0mm
- moved TP1 251.4 mm to (185.9, 90.1)
- moved TP4 246.6 mm to (185.9, 101.0)
- moved TP5 246.6 mm to (185.9, 104.1)
- moved TP2 246.6 mm to (185.9, 94.9)
- moved TP3 246.6 mm to (185.9, 98.0)
- moved J1 244.9 mm to (146.7, 116.1)
- moved J2 237.3 mm to (124.2, 113.1)
- moved F1 235.3 mm to (136.3, 108.9)
- moved C17 230.1 mm to (173.4, 118.1), turned to 90 degrees
- moved C19 230.0 mm to (176.4, 118.1), turned to 90 degrees
- moved C1 224.7 mm to (136.6, 121.4)
- moved U1 223.1 mm to (124.3, 102.1)
- moved Q2 222.3 mm to (164.0, 116.7), turned to 90 degrees
- moved Q3 221.4 mm to (168.5, 116.7), turned to 90 degrees
- moved C10 219.7 mm to (139.6, 79.9)
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Other:
- board outline added: 149.8 x 61.2 mm

Commit message: 20260606
Parts:
- moved R15 24.3 mm to (192.3, 43.8)
- moved R20 24.3 mm to (192.3, 48.8)
- moved C9 17.3 mm to (144.8, 74.1), turned to 90 degrees
- moved C10 12.0 mm to (149.2, 72.7), turned to 90 degrees
- moved C6 9.39 mm to (128.8, 102.5)
- moved C11 8.85 mm to (147.0, 87.8), turned to -90 degrees
- moved C8 7.40 mm to (194.2, 69.7), turned to -90 degrees
- moved C7 6.81 mm to (191.2, 71.1), turned to -90 degrees
- moved LED5-GREEN1 5.83 mm to (146.6, 100.0)
- moved U5 5.83 mm to (146.4, 95.5)
- turned U1 to -90 degrees

Commit message: 20260606
Parts:
- moved R19 2.63 mm to (213.0, 92.1), turned to -90 degrees
Changed lines of the file:
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@@
 	(footprint "Resistor_SMD:R_0805_2012Metric"
 		(layer "F.Cu")
-		(at 211.6325 89.84)
+		(at 213 92.0875 -90)
 		(descr "Resistor SMD 0805 (2012 Metric), square (rectangular) end terminal, IPC-7351 nominal, (Body size source: IPC-SM-782 page 72, https://www.pcb-3d.com/wordpress/wp-content/uploads/ipc-sm-782a_amendment_1_and_2.pdf), generated with kicad-footprint-generator")
 		(tags "resistor")
 		(property "Reference" "R19"
-			(at 0 -1.65 0)
+			(at 0 -1.65 90)
 			(layer "F.SilkS")
 			(effects
@@
 		)
 		(property "Value" "10K"
-			(at 0 1.65 0)
+			(at 0 1.65 90)
 			(layer "F.Fab")
 			(effects
@@
 		)
 		(property "Datasheet" "~"
-			(at 0 0 0)
+			(at 0 0 90)
 			(layer "F.Fab")
 			(hide yes)
@@
 		)
 		(property "Description" "Resistor"
-			(at 0 0 0)
+			(at 0 0 90)
 			(layer "F.Fab")
 			(hide yes)
@@
 		(attr smd)
 		(fp_line
-			(start -0.227064 -0.735)
-			(end 0.227064 -0.735)
+			(start -0.227064 0.735)
+			(end 0.227064 0.735)
 			(stroke
 				(width 0.12)
@@
 		)
 		(fp_line
-			(start -0.227064 0.735)
-			(end 0.227064 0.735)
+			(start -0.227064 -0.735)
+			(end 0.227064 -0.735)
 			(stroke
 				(width 0.12)
@@
 		)
 		(fp_text user "${REFERENCE}"
-			(at 0 0 0)
+			(at 0 0 90)
 			(layer "F.Fab")
 			(effects
@@
 		)
 		(pad "1" smd roundrect
-			(at -0.9125 0)
+			(at -0.9125 0 270)
 			(size 1.025 1.4)
 			(layers "F.Cu" "F.Mask" "F.Paste")
@@
 		)
 		(pad "2" smd roundrect
-			(at 0.9125 0)
+			(at 0.9125 0 270)
 			(size 1.025 1.4)
 			(layers "F.Cu" "F.Mask" "F.Paste")

Commit message: 20260607
Parts:
- moved R15 33.6 mm to (194.0, 77.3), turned to -90 degrees
- moved R20 28.6 mm to (192.0, 77.3), turned to 90 degrees

Commit message: 20260513
Parts:
- added C21: 1u, Capacitor_SMD:C_0805_2012Metric, F.Cu at (165.2, 78.7)
- added C22: 10n, Capacitor_SMD:C_0805_2012Metric, F.Cu at (179.8, 82.8)
- moved R25 91.7 mm to (183.7, 76.5), turned to 180 degrees
- moved R24 91.2 mm to (182.0, 71.0)
- moved R35 90.6 mm to (180.1, 76.5), turned to 180 degrees
- moved U7 86.6 mm to (181.9, 73.8)
- moved C15 85.7 mm to (179.1, 73.6), turned to -90 degrees
- moved R28 71.5 mm to (179.0, 90.0)
- moved R27 69.0 mm to (183.4, 82.8), turned to 180 degrees
- moved U2 62.8 mm to (183.3, 85.4)
- moved R26 62.5 mm to (175.0, 90.0)
- moved C16 60.6 mm to (175.0, 86.2)
- moved C18 51.6 mm to (165.3, 88.7)
- moved C20 51.6 mm to (165.3, 91.7)
- moved R29 51.6 mm to (160.9, 85.5)
- moved R30 51.6 mm to (160.9, 88.5)
- moved R31 51.6 mm to (160.9, 91.5)
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Connections:
- MK1 pad OUT: Net-(U2-IN+) -> Net-(C22-Pad1)
- R28 pad 2: Net-(U2-IN+) -> Net-(C22-Pad1)
- R30 pad 2: GND -> Net-(C21-Pad1)
Other:
- board size 149.8 x 61.2 mm -> 149.8 x 55.8 mm
