File: Projects/Tutorial03-ESP32-IoT-4-layer-PCB/Tutorial03-ESP32-IoT-4-layer-PCB.kicad_pcb (KiCad board)
At the start: 4 copper layers, 149.8 x 55.8 mm, 88 parts, among them J1 SS-52400-002, J2 B2B-PH-SM4-TB, J3 GSD090012SEU, J4 Conn_01x04_Pin, J5 Conn_01x05_Pin, Q1 TEMT6000X01, Q2 BC817, Q3 BC817, U1 MCP73871, U2 MAX4466EXK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

Commit message: 20260614
Parts:
- moved R3 64.3 mm to (186.2, 103.0), turned to 90 degrees
- moved F1 61.8 mm to (183.2, 101.5), turned to 90 degrees
- moved R4 59.0 mm to (180.5, 102.1), turned to 90 degrees
- moved C1 57.3 mm to (177.7, 102.2), turned to 90 degrees
- moved J1 50.1 mm to (181.9, 112.0)
- moved C17 47.9 mm to (167.9, 65.1), turned to -90 degrees
- moved C19 44.8 mm to (167.9, 68.7)
- moved S1 41.8 mm to (171.4, 64.6), turned to 180 degrees
- moved S2 39.5 mm to (171.4, 67.2), turned to 0 degrees
- moved R32 37.8 mm to (171.5, 69.6), turned to 0 degrees
- moved Q2 36.9 mm to (168.2, 74.5)
- moved Q3 33.7 mm to (172.0, 77.6), turned to -90 degrees
- moved R34 32.2 mm to (171.8, 74.4), turned to 0 degrees
- moved R33 29.0 mm to (168.3, 77.6), turned to 180 degrees
- moved MK1 23.7 mm to (170.8, 90.5), turned to 90 degrees
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
Commit message: 20260620
Parts:
- LED5G1: renamed from LED5-GREEN1; footprint Project-Footprints:T491A -> Project-Footprints:LEDC2012X120N
- moved R5 62.3 mm to (170.1, 107.0)
- moved R2 61.9 mm to (170.1, 100.7)
- moved C9 61.1 mm to (186.7, 95.4), turned to -90 degrees
- moved R6 59.7 mm to (170.1, 104.9)
- moved R1 57.1 mm to (161.1, 106.8), turned to 180 degrees
- moved J2 56.4 mm to (165.7, 110.9)
- moved C10 54.3 mm to (183.8, 94.1), turned to -90 degrees
- moved U1 51.2 mm to (165.6, 105.3)
- moved C6 50.7 mm to (170.1, 102.8)
- moved U4 50.6 mm to (182.2, 89.5)
- moved LED1R1 50.1 mm to (166.2, 100.7), turned to -90 degrees
- moved R9 49.5 mm to (163.9, 100.8), turned to 90 degrees
- moved R7 49.4 mm to (161.1, 102.7), turned to 180 degrees
- moved R8 49.0 mm to (161.1, 104.7), turned to 180 degrees
- moved C11 47.9 mm to (179.5, 94.1)
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- renumbered LED1-RED1 to LED1R1, LED2-GREEN1 to LED2G1, LED3-BLUE1 to LED3B1, LED6-RED1 to LED6R1

Commit message: 20260625
Parts:
- moved C4 20.3 mm to (122.0, 103.7), turned to -90 degrees
- moved R10 19.6 mm to (137.2, 99.2), turned to 180 degrees
- moved C3 19.4 mm to (137.0, 103.7)
- moved VR1 18.8 mm to (129.5, 102.5)
- moved C2 14.2 mm to (134.0, 105.0)
- moved C5 13.5 mm to (125.0, 105.0), turned to -90 degrees
- moved LED2R1 12.4 mm to (133.5, 99.0), turned to 180 degrees
- renumbered LED2-RED1 to LED2R1
Changed lines of the file:
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@@
 	(net 36 "/ESP-32-C3-02/GPIO18")
 	(net 37 "/ESP-32-C3-02/GPIO8")
-	(net 38 "Net-(LED2-RED1-K)")
+	(net 38 "Net-(LED2R1-K)")
 	(net 39 "Net-(LED5G1-K)")
 	(net 40 "Net-(LED6R1-K)")
@@
 	(footprint "Project-Footprints:T491A"
 		(layer "F.Cu")
-		(at 128.04 86.49 90)
+		(at 137 103.7 90)
 		(descr "T491A-1")
 		(tags "Capacitor Polarised")
 		(property "Reference" "C3"
-			(at 0 0 90)
+			(at -4.3 0 180)
 			(layer "F.SilkS")
 			(effects
@@
 	(footprint "Project-Footprints:VREG_LM1117MPX-3.3"
 		(layer "F.Cu")
-		(at 120.79 85.8 90)
+		(at 129.5 102.5 90)
 		(descr "Power Management IC’s LM117MPX-3.3/NOPB")
 		(property "Reference" "VR1"
-			(at -0.025 -4.754 90)
+			(at -5.5 0 180)
 			(layer "F.SilkS")
 			(effects
@@
 	(footprint "Project-Footprints:LEDC2012X120N"
 		(layer "F.Cu")
-		(at 122.215 94.01)
+		(at 133.5 99.05 180)
 		(descr "LTST-C170TBKT")
 		(tags "LED")
-		(property "Reference" "LED2-RED1"
-			(at 0 0 0)
+		(property "Reference" "LED2R1"
+			(at 1.25 2.05 0)
 			(layer "F.SilkS")
 			(effects
@@
 		)
 		(property "Height" "1.2"
-			(at 0 0 0)
+			(at 0 0 180)
 			(unlocked yes)
 			(layer "F.Fab")
@@
 		)
 		(property "Manufacturer_Name" "Lite-On"
-			(at 0 0 0)
+			(at 0 0 180)
 			(unlocked yes)
 			(layer "F.Fab")
@@
 		)
 		(property "Manufacturer_Part_Number" "LTST-C170KRKT"
-			(at 0 0 0)
+			(at 0 0 180)
 			(unlocked yes)
 			(layer "F.Fab")
@@
 		)
 		(property "Mouser Part Number" "859-LTST-C170KRKT"
-			(at 0 0 0)
+			(at 0 0 180)
 			(unlocked yes)
 			(layer "F.Fab")
@@
 		)
 		(property "Mouser Price/Stock" "https://www.mouser.co.uk/ProductDetail/Lite-On/LTST-C170KRKT?qs=NUb82WqeCyrVOID%2Fxt4rgA%3D%3D"
-			(at 0 0 0)
+			(at 0 0 180)
 			(unlocked yes)
 			(layer "F.Fab")
@@
 		)
 		(property "Arrow Part Number" "LTST-C170KRKT"
-			(at 0 0 0)
+			(at 0 0 180)
 			(unlocked yes)
 			(layer "F.Fab")
@@
 		)
 		(property "Arrow Price/Stock" "https://www.arrow.com/en/products/ltst-c170krkt/lite-on-technology?utm_currency=USD&region=nac"
-			(at 0 0 0)
+			(at 0 0 180)
 			(unlocked yes)
 			(layer "F.Fab")
@@
 		(attr smd)
 		(fp_line
-			(start -1.75 -1.05)
-			(end -1.75 1.05)
+			(start 0.9 -1.05)
+			(end -1.75 -1.05)
 			(stroke
 				(width 0.2)
@@
 		)
 		(fp_line
-			(start 0.9 -1.05)
-			(end -1.75 -1.05)
+			(start -1.75 -1.05)
+			(end -1.75 1.05)
 			(stroke
 				(width 0.2)
@@
 		)
 		(fp_line
-			(start -1.85 -1.15)
-			(end 1.85 -1.15)
+			(start 1.85 1.15)
+			(end -1.85 1.15)
 			(stroke
 				(width 0.05)
@@
 		)
 		(fp_line
-			(start -1.85 1.15)
-			(end -1.85 -1.15)
+			(start 1.85 -1.15)
+			(end 1.85 1.15)
 			(stroke
 				(width 0.05)
@@
 		)
 		(fp_line
-			(start 1.85 -1.15)
-			(end 1.85 1.15)
+			(start -1.85 1.15)
+			(end -1.85 -1.15)
 			(stroke
 				(width 0.05)
@@
 		)
 		(fp_line
-			(start 1.85 1.15)
-			(end -1.85 1.15)
+			(start -1.85 -1.15)
+			(end 1.85 -1.15)
 			(stroke
 				(width 0.05)
@@
 		)
 		(fp_line
-			(start -1 -0.625)
-			(end 1 -0.625)
+			(start 1 0.625)
+			(end -1 0.625)
 			(stroke
 				(width 0.1)
@@
 		)
 		(fp_line
-			(start -1 -0.208)
-			(end -0.583 -0.625)
+			(start 1 -0.625)
+			(end 1 0.625)
 			(stroke
 				(width 0.1)
@@
 		)
 		(fp_line
-			(start 1 -0.625)
-			(end 1 0.625)
+			(start -1 -0.208)
+			(end -0.583 -0.625)
 			(stroke
 				(width 0.1)
@@
 		)
 		(fp_line
-			(start 1 0.625)
-			(end -1 0.625)
+			(start -1 -0.625)
+			(end 1 -0.625)
 			(stroke
 				(width 0.1)
@@
 		)
 		(pad "1" smd rect
-			(at -0.9 0)
+			(at -0.9 0 180)
 			(size 1 1.4)
 			(layers "F.Cu" "F.Mask" "F.Paste")
-			(net 38 "Net-(LED2-RED1-K)")
+			(net 38 "Net-(LED2R1-K)")
 			(pinfunction "K")
 			(pintype "passive")
 		)
 		(pad "2" smd rect
-			(at 0.9 0)
+			(at 0.9 0 180)
 			(size 1 1.4)
 			(layers "F.Cu" "F.Mask" "F.Paste")
@@
 	(footprint "Project-Footprints:T491A"
 		(layer "F.Cu")
-		(at 132.69 86.49 90)
+		(at 122 103.69 -90)
 		(descr "T491A-1")
 		(tags "Capacitor Polarised")
 		(property "Reference" "C4"
-			(at 0 0 90)
+			(at 4.31 0 180)
 			(layer "F.SilkS")
 			(effects
@@
 		)
 		(fp_line
-			(start 3.01 -1.8)
-			(end 3.01 1.8)
+			(start -3.01 1.8)
+			(end -3.01 -1.8)
 			(stroke
 				(width 0.05)
@@
 		)
 		(fp_line
-			(start -3.01 -1.8)
-			(end 3.01 -1.8)
+			(start 3.01 1.8)
+			(end -3.01 1.8)
 			(stroke
 				(width 0.05)
@@
 		)
 		(fp_line
-			(start 3.01 1.8)
-			(end -3.01 1.8)
+			(start -3.01 -1.8)
+			(end 3.01 -1.8)
 			(stroke
 				(width 0.05)
@@
 		)
 		(fp_line
-			(start -3.01 1.8)
-			(end -3.01 -1.8)
+			(start 3.01 -1.8)
+			(end 3.01 1.8)
 			(stroke
 				(width 0.05)
@@
 		)
 		(fp_line
-			(start 1.6 -0.8)
-			(end 1.6 0.8)
+			(start -1.6 0.8)
+			(end -1.6 -0.8)
 			(stroke
 				(width 0.2)
@@
 		)
 		(fp_line
-			(start -1.6 -0.8)
-			(end 1.6 -0.8)
+			(start 1.6 0.8)
+			(end -1.6 0.8)
 			(stroke
 				(width 0.2)
@@
 		)
 		(fp_line
-			(start 1.6 0.8)
-			(end -1.6 0.8)
+			(start -1.6 -0.8)
+			(end 1.6 -0.8)
 			(stroke
 				(width 0.2)
@@
 		)
 		(fp_line
-			(start -1.6 0.8)
-			(end -1.6 -0.8)
+			(start 1.6 -0.8)
+			(end 1.6 0.8)
 			(stroke
 				(width 0.2)
@@
 		)
 		(pad "1" smd rect
-			(at -1.31 0 180)
+			(at -1.31 0)
 			(size 1.23 1.8)
 			(layers "F.Cu" "F.Mask" "F.Paste")
@@
 		)
 		(pad "2" smd rect
-			(at 1.31 0 180)
+			(at 1.31 0)
 			(size 1.23 1.8)
 			(layers "F.Cu" "F.Mask" "F.Paste")
@@
 	(footprint "Capacitor_SMD:C_0805_2012Metric"
 		(layer "F.Cu")
-		(at 130.2 92.5 90)
+		(at 125 105 -90)
 		(descr "Capacitor SMD 0805 (2012 Metric), square (rectangular) end terminal, IPC-7351 nominal, (Body size source: IPC-SM-782 page 76, https://www.pcb-3d.com/wordpress/wp-content/uploads/ipc-sm-782a_amendment_1_and_2.pdf, https://docs.google.com/spreadsheets/d/1BsfQQcO9C6DZCsRaXUlFlo91Tg2WpOkGARC1WS5S8t0/edit?usp=sharing), generated with kicad-footprint-generator")
 		(tags "capacitor")
 		(property "Reference" "C5"
-			(at 0 -1.68 90)
+			(at 3 0 180)
 			(layer "F.SilkS")
 			(effects
@@
 		(attr smd)
 		(fp_line
-			(start -0.261252 -0.735)
-			(end 0.261252 -0.735)
+			(start -0.261252 0.735)
+			(end 0.261252 0.735)
 			(stroke
 				(width 0.12)
@@
 		)
 		(fp_line
-			(start -0.261252 0.735)
-			(end 0.261252 0.735)
+			(start -0.261252 -0.735)
+			(end 0.261252 -0.735)
 			(stroke
 				(width 0.12)
@@
 		)
 		(pad "1" smd roundrect
-			(at -0.95 0 90)
+			(at -0.95 0 270)
 			(size 1 1.45)
 			(layers "F.Cu" "F.Mask" "F.Paste")
@@
 		)
 		(pad "2" smd roundrect
-			(at 0.95 0 90)
+			(at 0.95 0 270)
 			(size 1 1.45)
 			(layers "F.Cu" "F.Mask" "F.Paste")
@@
 	(footprint "Capacitor_SMD:C_0805_2012Metric"
 		(layer "F.Cu")
-		(at 127.19 92.5 90)
+		(at 133.96 105.01 90)
 		(descr "Capacitor SMD 0805 (2012 Metric), square (rectangular) end terminal, IPC-7351 nominal, (Body size source: IPC-SM-782 page 76, https://www.pcb-3d.com/wordpress/wp-content/uploads/ipc-sm-782a_amendment_1_and_2.pdf, https://docs.google.com/spreadsheets/d/1BsfQQcO9C6DZCsRaXUlFlo91Tg2WpOkGARC1WS5S8t0/edit?usp=sharing), generated with kicad-footprint-generator")
 		(tags "capacitor")
 		(property "Reference" "C2"
-			(at 0 -1.68 90)
+			(at -2.99 0.04 180)
 			(layer "F.SilkS")
 			(effects
@@
 	(footprint "Resistor_SMD:R_0805_2012Metric"
 		(layer "F.Cu")
-		(at 117.635 98.91)
+		(at 137.25 99.25 180)
 		(descr "Resistor SMD 0805 (2012 Metric), square (rectangular) end terminal, IPC-7351 nominal, (Body size source: IPC-SM-782 page 72, https://www.pcb-3d.com/wordpress/wp-content/uploads/ipc-sm-782a_amendment_1_and_2.pdf), generated with kicad-footprint-generator")
 		(tags "resistor")
 		(property "Reference" "R10"
-			(at 0 -1.65 0)
+			(at 0 2.25 180)
 			(layer "F.SilkS")
 			(effects
@@
 		(attr smd)
 		(fp_line
-			(start -0.227064 -0.735)
-			(end 0.227064 -0.735)
+			(start -0.227064 0.735)
+			(end 0.227064 0.735)
 			(stroke
 				(width 0.12)
@@
 		)
 		(fp_line
-			(start -0.227064 0.735)
-			(end 0.227064 0.735)
+			(start -0.227064 -0.735)
+			(end 0.227064 -0.735)
 			(stroke
 				(width 0.12)
@@
 		)
 		(pad "1" smd roundrect
-			(at -0.9125 0)
+			(at -0.9125 0 180)
 			(size 1.025 1.4)
 			(layers "F.Cu" "F.Mask" "F.Paste")
@@
 		)
 		(pad "2" smd roundrect
-			(at 0.9125 0)
+			(at 0.9125 0 180)
 			(size 1.025 1.4)
 			(layers "F.Cu" "F.Mask" "F.Paste")
 			(roundrect_rratio 0.243902)
-			(net 38 "Net-(LED2-RED1-K)")
+			(net 38 "Net-(LED2R1-K)")
 			(pintype "passive")
 		)
@@
 	)
 	(gr_line
-		(start 72.75 61.25)
-		(end 72.75 117)
+		(start 179 66.75)
+		(end 179 61.25)
 		(stroke
 			(width 0.05)
-			(type solid)
+			(type default)
 		)
 		(layer "Edge.Cuts")
 	)
 	(gr_line
-		(start 72.75 117)
-		(end 222.5 117)
+		(start 72.75 61.25)
+		(end 72.75 117)
 		(stroke
 			(width 0.05)
-			(type default)
+			(type solid)
 		)
 		(layer "Edge.Cuts")
 	)
 	(gr_line
-		(start 179 61.25)
-		(end 72.75 61.25)
+		(start 222.5 117)
+		(end 222.5 66.75)
 		(stroke
 			(width 0.05)
-			(type default)
+			(type solid)
 		)
 		(layer "Edge.Cuts")
 	)
 	(gr_line
-		(start 179 66.75)
-		(end 179 61.25)
+		(start 195 66.75)
+		(end 179 66.75)
 		(stroke
 			(width 0.05)
@@
 	)
 	(gr_line
-		(start 195 66.75)
-		(end 179 66.75)
+		(start 222.5 66.75)
+		(end 195 66.75)
 		(stroke
 			(width 0.05)
@@
 	)
 	(gr_line
-		(start 222.5 66.75)
-		(end 195 66.75)
+		(start 72.75 117)
+		(end 222.5 117)
 		(stroke
 			(width 0.05)
@@
 	)
 	(gr_line
-		(start 222.5 117)
-		(end 222.5 66.75)
+		(start 179 61.25)
+		(end 72.75 61.25)
 		(stroke
 			(width 0.05)
-			(type solid)
+			(type default)
 		)
 		(layer "Edge.Cuts")

Commit message: 20260626
Parts:
- added 2.5: MountingHole_2.5mm, MountingHole:MountingHole_2.5mm, F.Cu at (179.2, 71.0)
- added 2.5: MountingHole_2.5mm, MountingHole:MountingHole_2.5mm, F.Cu at (179.2, 115.6)
- added 2.5: MountingHole_2.5mm, MountingHole:MountingHole_2.5mm, F.Cu at (96.8, 65.4)
- added REF**: MountingHole_2.5mm, MountingHole:MountingHole_2.5mm, F.Cu at (97.0, 115.6)
- moved C6 50.7 mm to (119.4, 104.2)
- moved J2 50.7 mm to (115.0, 112.2)
- moved LED2G1 50.7 mm to (110.2, 99.3)
- moved LED3B1 50.7 mm to (110.2, 101.8)
- moved U1 50.7 mm to (114.9, 106.7)
- moved LED1R1 50.7 mm to (115.5, 102.0)
- moved R1 50.7 mm to (110.4, 108.2)
- moved R2 50.7 mm to (119.4, 102.1)
- moved R5 50.7 mm to (119.4, 108.3)
- moved R6 50.7 mm to (119.4, 106.2)
- moved R7 50.7 mm to (110.4, 104.1)
- moved R8 50.7 mm to (110.4, 106.1)
- moved R9 50.7 mm to (113.3, 102.2)
- moved C1 50.0 mm to (128.2, 105.3)
- moved F1 50.0 mm to (133.2, 103.8)
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Other:
- board size 149.8 x 55.8 mm -> 88 x 55.8 mm

Commit message: 20260626
Routing:
- added copper zone on In2.Cu, net GND
Changed lines of the file:
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@@
 		(layer "Edge.Cuts")
+	)
+	(zone
+		(net 1)
+		(net_name "GND")
+		(layer "In2.Cu")
+		(name "GND")
+		(hatch edge 0.5)
+		(connect_pads
+			(clearance 0.5)
+		)
+		(min_thickness 0.25)
+		(filled_areas_thickness no)
+		(fill
+			(thermal_gap 0.5)
+			(thermal_bridge_width 0.5)
+		)
+		(polygon
+			(pts
+				(xy 86.8 60.2) (xy 86.8 120.2) (xy 186.2 120.2) (xy 186.6 60.2)
+			)
+		)
 	)
 	(group ""

Commit message: 20260628
Parts:
- moved U5 13.5 mm to (132.6, 102.7), turned to -90 degrees
- moved C1 9.36 mm to (137.6, 104.8), turned to 90 degrees
- moved F1 6.88 mm to (126.3, 103.2)
- moved R3 6.08 mm to (139.6, 110.3)
- moved R4 3.78 mm to (126.8, 106.7), turned to -90 degrees
Routing:
- added copper zone on In1.Cu, net +3.3V
- added copper zone on In1.Cu, net /+5V_USB
- added copper zone on In1.Cu, net /VBUS
