File: Projects/Tutorial03-ESP32-IoT-4-layer-PCB/Tutorial03-ESP32-IoT-4-layer-PCB.kicad_pcb (KiCad board)
At the start: 4 copper layers, 88 x 55.8 mm, 92 parts, among them J1 SS-52400-002, J2 B2B-PH-SM4-TB, J3 GSD090012SEU, J4 Conn_01x04_Pin, J5 Conn_01x05_Pin, Q1 TEMT6000X01, Q2 BC817, Q3 BC817, U1 MCP73871, U2 MAX4466EXK, U3 ESP32-C3-WROOM-02-H4, U4 CP2102N-Axx-xQFN20, U5 USBLC6-2SC6, U6 W25Q32JVSSIQ, U7 BME280

Commit message: 20260704
Parts:
- moved R18 14.3 mm to (126.9, 99.0), turned to 0 degrees
- moved LED6R1 12.4 mm to (126.7, 94.7), turned to 180 degrees
- moved R16 11.6 mm to (126.9, 97.0), turned to 180 degrees
- moved R12 9.99 mm to (135.5, 100.4), turned to 90 degrees
- moved C9 9.56 mm to (130.5, 91.1)
- moved R13 7.63 mm to (136.2, 97.7), turned to 0 degrees
- moved LED5G1 6.55 mm to (126.7, 92.3), turned to 180 degrees
- moved U4 6.27 mm to (131.8, 96.9), turned to 90 degrees
- moved C11 5.24 mm to (136.2, 95.6), turned to 0 degrees
- moved R11 3.66 mm to (136.2, 93.6), turned to 180 degrees
- moved C10 3.59 mm to (133.4, 92.4)
- moved C2 0.56 mm to (108.5, 86.9)
- moved C3 0.56 mm to (105.4, 88.2)
- moved C4 0.56 mm to (120.4, 88.2)
- moved C5 0.56 mm to (117.4, 86.9)
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Routing:
- net /VBAT: track 0.00 -> 5.89 mm
- net GND: vias 0 -> 5
- net /VBUS: vias 0 -> 2
- net /+5V_USB: vias 0 -> 3
- added copper zone on F.Cu, net /+5V_USB
- added copper zone on F.Cu, net /VBAT
- added copper zone on F.Cu, net /VBUS
- added copper zone on F.Cu, net GND

Commit message: 20260711
Parts:
- moved J4 50.1 mm to (132.2, 64.7), turned to -90 degrees
- moved R33 14.7 mm to (135.2, 82.5), turned to -90 degrees
- moved Q2 13.1 mm to (132.2, 82.6), turned to 180 degrees
- moved C17 12.9 mm to (124.4, 78.8)
- moved C19 12.9 mm to (124.4, 82.4)
- moved R32 12.9 mm to (128.0, 83.3)
- moved S1 12.9 mm to (127.9, 78.3)
- moved S2 12.9 mm to (127.9, 80.9)
- moved Q3 10.6 mm to (135.2, 78.8), turned to 0 degrees
- moved R25 8.86 mm to (132.9, 68.3), turned to -90 degrees
- moved R34 8.19 mm to (132.1, 79.0), turned to 90 degrees
- moved U7 8.05 mm to (128.2, 68.2), turned to 90 degrees
- moved C15 7.81 mm to (125.6, 68.3), turned to 90 degrees
- moved C7 7.10 mm to (149.4, 65.6)
- moved C8 7.10 mm to (152.4, 64.2)
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Connections:
- J4 pad 2: /ESP-32-C3-02/SDA -> /ESP-32-C3-02/SCL
- J4 pad 3: /ESP-32-C3-02/SCL -> /ESP-32-C3-02/SDA
Routing:
- net /ESP-32-C3-02/SCL: track 0.00 -> 52.5 mm
- net /ESP-32-C3-02/SDA: track 0.00 -> 34.4 mm
- net /ESP-32-C3-02/USB_D+: track 0.00 -> 3.15 mm
- net /ESP-32-C3-02/USB_D-: track 0.00 -> 3.12 mm
- net /USB_DP: track 0.00 -> 3.00 mm
- net /USB_DN: track 0.00 -> 2.97 mm
- net Net-(U7-SDO): track 0.00 -> 2.71 mm
- net GND: vias 5 -> 22
- net /VBUS: vias 2 -> 3
