File: Projects/Tutorial03-ESP32-IoT-4-layer-PCB/user_interface.kicad_sch (KiCad schematic)
At the start: 11 parts, among them J4 Conn_01x04_Pin, J5 Conn_01x05_Pin, Q2 BC817, Q3 BC817

Commit message: 20260711
Connections:
- net SCL: now also J4.2 (Pin_2); no longer J4.3 (Pin_3)
- net SDA: now also J4.3 (Pin_3); no longer J4.2 (Pin_2)
